Commit message: Updated xarm ros2 ws with init compatibility test

File: xarm_ros2/xarm_description/urdf/common/common.link.xacro (robot description, xacro)
@@ -75,5 +75,10 @@
     <xacro:property name="mass_type" value="-1" />
     <xacro:property name="model_type" value="-1" />
-    <xacro:property name="_model1300" value="${model1300}" />
+    <xacro:if value="${model1300}">
+      <xacro:property name="model_num" value="1300" />
+    </xacro:if>
+    <xacro:unless value="${model1300}">
+      <xacro:property name="model_num" value="-1" />
+    </xacro:unless>
     <!-- parse model_type and mass_type from robot_sn -->
     <xacro:if value="${robot_sn_len >= 14 and (robot_sn[0] == 'X' or robot_sn[0] == 'L' or robot_sn[0] == 'F')}">
@@ -102,5 +107,4 @@
         </xacro:if>
       </xacro:if>
-      <!-- <xacro:property name="model_type" value="${9 if robot_sn[0] == 'L' else 5 if robot_sn[1] == 'F' else 6 if robot_sn[1] == 'I' else 7 if robot_sn[1] == 'S' else -1}" /> -->
       <xacro:property name="model_num" value="${int(robot_sn[2:6])}" />
       <xacro:if value="${model_num == 1250}">
@@ -112,7 +116,4 @@
         <xacro:property name="mass_type" value="1" />
       </xacro:if>
-      <xacro:if value="${model_num >= 1300}">
-        <xacro:property name="_model1300" value="true" />
-      </xacro:if>
       <xacro:property name="is_num" value="${robot_sn[8] == '0' or robot_sn[8] == '1' or robot_sn[8] == '2' or robot_sn[8] == '3' or robot_sn[8] == '4' or robot_sn[8] == '5' or robot_sn[8] == '6' or robot_sn[8] == '7' or robot_sn[8] == '8' or robot_sn[8] == '9'}" />
       <xacro:if value="${is_num}">
@@ -134,5 +135,4 @@
         </xacro:unless>
       </xacro:unless>
-      <!-- <xacro:property name="hd_type" value="${robot_sn[11] if robot_sn[11] == 'B' or robot_sn[11] == 'L' or robot_sn[11] == 'X' or robot_sn[11] == 'D' else robot_sn[15] if robot_sn_len >= 16 and robot_sn[14] == '_' else ''}" /> -->
       <xacro:if value="${hd_type == 'B'}">
         <xacro:if value="${date_int >= 2004}">
@@ -142,5 +142,4 @@
           <xacro:property name="mass_type" value="1" />
         </xacro:unless>
-        <!-- <xacro:property name="mass_type" value="${11 if date_int >= 2004 else 1}" /> -->
       </xacro:if>
       <xacro:unless value="${hd_type == 'B'}">
@@ -149,5 +148,5 @@
           <xacro:property name="mass_type" value="2" />
         </xacro:if>
-        <xacro:if value="${hd_type == 'X'}">
+        <xacro:if value="${hd_type == 'A'}">
           <xacro:property name="mass_type" value="3" />
         </xacro:if>
@@ -155,74 +154,76 @@
           <xacro:property name="mass_type" value="4" />
         </xacro:if>
-        <!-- <xacro:property name="mass_type" value="${2 if hd_type == 'L' else 3 if hd_type == 'X' else 4 if hd_type == 'D' else 1}" /> -->
-      </xacro:unless>
-    </xacro:if>
-    <!-- update xarm5 inertia params filename -->
-    <xacro:if value="${dof == 5}">
-      <xacro:if value="${model_type == 5}">
-        <xacro:if value="${mass_type == 1}">
-          <xacro:property name="inertial_params_filename" value="xarm5_type5_HT_BR"/>
-        </xacro:if>
-        <xacro:if value="${mass_type == 2}">
-          <xacro:property name="inertial_params_filename" value="xarm5_type5_HT_LD"/>
-        </xacro:if>
-        <xacro:if value="${mass_type == 11}">
-          <xacro:property name="inertial_params_filename" value="xarm5_type5_HT_BR2"/>
-        </xacro:if>
-      </xacro:if>
-    </xacro:if>
-    <xacro:if value="${dof == 6}">
-      <!-- update uf850 inertia params filename -->
-      <xacro:if value="${robot_type == 'uf850'}">
-        <xacro:if value="${model_type == 12}">
-          <xacro:property name="inertial_params_filename" value="xarm6_type12_HT_LDBR2"/>
-        </xacro:if>
-      </xacro:if>
-      <!-- update lite6 inertia params filename -->
-      <xacro:if value="${robot_type == 'lite'}">
-        <xacro:if value="${model_type == 9}">
-          <xacro:property name="inertial_params_filename" value="xarm6_type9_HT_BR2"/>
-        </xacro:if>
-      </xacro:if>
-      <!-- update xarm6 inertia params filename -->
-      <xacro:unless value="${robot_type == 'lite' or robot_type == 'uf850'}">
-        <xacro:if value="${model_type == 6}">
+      </xacro:unless>
+      <!-- update xarm5 inertia params filename -->
+      <xacro:if value="${dof == 5}">
+        <xacro:if value="${model_type == 5}">
           <xacro:if value="${mass_type == 1}">
-            <xacro:property name="inertial_params_filename" value="xarm6_type6_HT_BR"/>
+            <xacro:property name="inertial_params_filename" value="xarm5_type5_HT_BR"/>
           </xacro:if>
           <xacro:if value="${mass_type == 2}">
-            <xacro:property name="inertial_params_filename" value="xarm6_type6_HT_LD"/>
+            <xacro:property name="inertial_params_filename" value="xarm5_type5_HT_LD"/>
           </xacro:if>
           <xacro:if value="${mass_type == 11}">
-            <xacro:property name="inertial_params_filename" value="xarm6_type6_HT_BR2"/>
-          </xacro:if>
-        </xacro:if>
-        <xacro:if value="${model_type == 8}">
-          <xacro:property name="inertial_params_filename" value="xarm6_type8_HT2_BR2"/>
-        </xacro:if>
-        <xacro:if value="${model_type == 11}">
-          <xacro:property name="inertial_params_filename" value="xarm6_type11_HT_LD"/>
-        </xacro:if>
-      </xacro:unless>
-    </xacro:if>
-    <!-- update xarm7 inertia params filename -->
-    <xacro:unless value="${dof == 5 or dof == 6}">
-      <xacro:if value="${model_type == 3}">
-        <xacro:property name="inertial_params_filename" value="xarm7_type3_YT_SP"/>
-      </xacro:if>
-      <xacro:if value="${model_type == 7}">
-        <xacro:if value="${mass_type == 1}">
-          <xacro:property name="inertial_params_filename" value="xarm7_type7_HT_BR"/>
-        </xacro:if>
-        <xacro:if value="${mass_type == 2}">
-          <xacro:property name="inertial_params_filename" value="xarm7_type7_HT_LD"/>
-        </xacro:if>
-        <xacro:if value="${mass_type == 11}">
-          <xacro:property name="inertial_params_filename" value="xarm7_type7_HT_BR2"/>
-        </xacro:if>
-      </xacro:if>
-    </xacro:unless>
+            <xacro:property name="inertial_params_filename" value="xarm5_type5_HT_BR2"/>
+          </xacro:if>
+        </xacro:if>
+      </xacro:if>
+      <xacro:if value="${dof == 6}">
+        <!-- update uf850 inertia params filename -->
+        <xacro:if value="${robot_type == 'uf850'}">
+          <xacro:if value="${model_type == 12}">
+            <xacro:property name="inertial_params_filename" value="xarm6_type12_HT_LDBR2"/>
+          </xacro:if>
+        </xacro:if>
+        <!-- update lite6 inertia params filename -->
+        <xacro:if value="${robot_type == 'lite'}">
+          <xacro:if value="${model_type == 9}">
+            <xacro:property name="inertial_params_filename" value="xarm6_type9_HT_BR2"/>
+          </xacro:if>
+        </xacro:if>
+        <!-- update xarm6 inertia params filename -->
+        <xacro:unless value="${robot_type == 'lite' or robot_type == 'uf850'}">
+          <xacro:if value="${model_type == 6}">
+            <xacro:if value="${mass_type == 1}">
+              <xacro:property name="inertial_params_filename" value="xarm6_type6_HT_BR"/>
+            </xacro:if>
+            <xacro:if value="${mass_type == 2}">
+              <xacro:property name="inertial_params_filename" value="xarm6_type6_HT_LD"/>
+            </xacro:if>
+            <xacro:if value="${mass_type == 3}">
+              <xacro:property name="inertial_params_filename" value="xarm6_type6_UJ_BR_2403"/>
+            </xacro:if>
+            <xacro:if value="${mass_type == 11}">
+              <xacro:property name="inertial_params_filename" value="xarm6_type6_HT_BR2"/>
+            </xacro:if>
+          </xacro:if>
+          <xacro:if value="${model_type == 8}">
+            <xacro:property name="inertial_params_filename" value="xarm6_type8_HT2_BR2"/>
+          </xacro:if>
+          <xacro:if value="${model_type == 11}">
+            <xacro:property name="inertial_params_filename" value="xarm6_type11_HT_LD"/>
+          </xacro:if>
+        </xacro:unless>
+      </xacro:if>
+      <!-- update xarm7 inertia params filename -->
+      <xacro:unless value="${dof == 5 or dof == 6}">
+        <xacro:if value="${model_type == 3}">
+          <xacro:property name="inertial_params_filename" value="xarm7_type3_YT_SP"/>
+        </xacro:if>
+        <xacro:if value="${model_type == 7}">
+          <xacro:if value="${mass_type == 1}">
+            <xacro:property name="inertial_params_filename" value="xarm7_type7_HT_BR"/>
+          </xacro:if>
+          <xacro:if value="${mass_type == 2}">
+            <xacro:property name="inertial_params_filename" value="xarm7_type7_HT_LD"/>
+          </xacro:if>
+          <xacro:if value="${mass_type == 11}">
+            <xacro:property name="inertial_params_filename" value="xarm7_type7_HT_BR2"/>
+          </xacro:if>
+        </xacro:if>
+      </xacro:unless>
+    </xacro:if>
     <xacro:property name="scope_parent_inertial_params_filename" value="${inertial_params_filename}" scope="parent"/>
-    <xacro:property name="scope_parent_model1300" value="${_model1300}" scope="parent"/>
+    <xacro:property name="scope_parent_model_num" value="${model_num}" scope="parent"/>
   </xacro:macro>
 </robot>

File: xarm_ros2/xarm_description/urdf/gripper/bio_gripper.ros2_control.xacro (robot description, xacro)
@@ -3,5 +3,5 @@
   <xacro:macro name="bio_gripper_ros2_control" params="prefix:=''
     ros2_control_plugin:='uf_robot_hardware/UFRobotFakeSystemHardware' ">
-    <ros2_control name="XArmGripperSystem" type="system">
+    <ros2_control name="BioGripperSystem" type="system">
       <hardware>
         <plugin>${ros2_control_plugin}</plugin>

File: xarm_ros2/xarm_description/urdf/gripper/bio_gripper.urdf.xacro (robot description, xacro)
@@ -32,6 +32,6 @@
         <mass value="0.012105" />
         <inertia
-          ixx="3.7322E-06" ixy="-4.1705E-06" ixz="4.0142E-06"
-          iyy="1.744E-05" iyz="-1.2237E-06" izz="1.7775E-05" />
+          ixx="3.7322E-06" ixy="4.1705E-06" ixz="-4.0142E-06"
+          iyy="1.744E-05" iyz="1.2237E-06" izz="1.7775E-05" />
       </inertial>
       <xacro:common_link_visual
@@ -58,6 +58,6 @@
         <mass value="0.012068" />
         <inertia
-          ixx="4.1413E-06" ixy="3.9682E-06" ixz="4.5734E-06"
-          iyy="1.6115E-05" iyz="1.6711E-06" izz="1.6032E-05" />
+          ixx="4.1413E-06" ixy="-3.9682E-06" ixz="-4.5734E-06"
+          iyy="1.6115E-05" iyz="-1.6711E-06" izz="1.6032E-05" />
       </inertial>
       <xacro:common_link_visual

File: xarm_ros2/xarm_description/urdf/lite6/lite6.urdf.xacro (robot description, xacro)
@@ -8,4 +8,5 @@
     joint5_lower_limit:=${-2.1642}  joint5_upper_limit:=${2.1642}
     joint6_lower_limit:=${-2.0*pi}  joint6_upper_limit:=${2.0*pi}
+    model_num:=0
     inertial_params_filename:='' kinematics_params_filename:='' "
     >

File: xarm_ros2/xarm_description/urdf/lite6/lite6_robot_macro.xacro (robot description, xacro)
@@ -12,4 +12,5 @@
     baud_checkset:=true
     default_gripper_baud:=2000000
+    model_num:=0
     inertial_params_filename:=''
     kinematics_params_filename:=''
@@ -45,4 +46,5 @@
         joint5_lower_limit="${-2.1642}" joint5_upper_limit="${2.1642}"
         joint6_lower_limit="${-pi*0.99}" joint6_upper_limit="${pi*0.99}"
+        model_num="${model_num}"
         inertial_params_filename="${inertial_params_filename}"
         kinematics_params_filename="${kinematics_params_filename}"
@@ -57,5 +59,5 @@
           baud_checkset="${baud_checkset}" default_gripper_baud="${default_gripper_baud}" />
       </xacro:if>
-      <xacro:lite6_urdf prefix="${prefix}"
+      <xacro:lite6_urdf prefix="${prefix}" model_num="${model_num}"
         inertial_params_filename="${inertial_params_filename}"
         kinematics_params_filename="${kinematics_params_filename}"

File: xarm_ros2/xarm_description/urdf/uf850/uf850.urdf.xacro (robot description, xacro)
@@ -8,5 +8,5 @@
     joint5_lower_limit:=${-2.1642}  joint5_upper_limit:=${2.1642}
     joint6_lower_limit:=${-2.0*pi}  joint6_upper_limit:=${2.0*pi}
-    model1300:=false
+    model_num:=0
     inertial_params_filename:='' kinematics_params_filename:='' "
     >

File: xarm_ros2/xarm_description/urdf/uf850/uf850_robot_macro.xacro (robot description, xacro)
@@ -13,5 +13,5 @@
     baud_checkset:='true'
     default_gripper_baud:=2000000
-    model1300:=false
+    model_num:=0
     inertial_params_filename:=''
     kinematics_params_filename:=''
@@ -47,5 +47,5 @@
         joint5_lower_limit="${-2.1642}" joint5_upper_limit="${2.1642}"
         joint6_lower_limit="${-pi*0.99}" joint6_upper_limit="${pi*0.99}"
-        model1300="${model1300}"
+        model_num="${model_num}"
         inertial_params_filename="${inertial_params_filename}"
         kinematics_params_filename="${kinematics_params_filename}"/>
@@ -59,5 +59,5 @@
           baud_checkset="${baud_checkset}" default_gripper_baud="${default_gripper_baud}" />
       </xacro:if>
-      <xacro:uf850_urdf prefix="${prefix}" model1300="${model1300}"
+      <xacro:uf850_urdf prefix="${prefix}" model_num="${model_num}"
         inertial_params_filename="${inertial_params_filename}"
         kinematics_params_filename="${kinematics_params_filename}"/>

File: xarm_ros2/xarm_description/urdf/xarm5/xarm5.urdf.xacro (robot description, xacro)
@@ -7,15 +7,15 @@
     joint4_lower_limit:=${-1.69297}  joint4_upper_limit:=${pi}
     joint5_lower_limit:=${-2.0*pi}  joint5_upper_limit:=${2.0*pi}
-    model1300:=false
+    model_num:=0
     inertial_params_filename:='' kinematics_params_filename:='' "
     >
     <!-- define property -->
-    <xacro:if value="${model1300}">
-      <xacro:property name="end_tool_visual_filename" value="end_tool/visual/end_tool_1300"/>
-      <xacro:property name="end_tool_collision_filename" value="end_tool/collision/end_tool_1300"/>
+    <xacro:if value="${model_num >= 1300}">
+      <xacro:property name="link5_visual" value="end_tool/visual/end_tool_1300"/>
+      <xacro:property name="link5_collision" value="end_tool/collision/end_tool_1300"/>
     </xacro:if>
-    <xacro:unless value="${model1300}">
-      <xacro:property name="end_tool_visual_filename" value="xarm5/visual/link5"/>
-      <xacro:property name="end_tool_collision_filename" value="end_tool/collision/end_tool"/>
+    <xacro:unless value="${model_num >= 1300}">
+      <xacro:property name="link5_visual" value="xarm5/visual/link5"/>
+      <xacro:property name="link5_collision" value="end_tool/collision/end_tool"/>
     </xacro:unless>
     <!-- load params and define property -->
@@ -167,10 +167,10 @@
         origin_rpy="0 0 0"/>
       <xacro:common_link_visual
-        mesh_filename="${end_tool_visual_filename}"
+        mesh_filename="${link5_visual}"
         origin_xyz="0 0 0"
         origin_rpy="0 0 0"
         material_name="${prefix}Silver" />
       <xacro:common_link_collision
-        mesh_filename="${end_tool_collision_filename}"
+        mesh_filename="${link5_collision}"
         origin_xyz="0 0 0"
         origin_rpy="0 0 0" />

File: xarm_ros2/xarm_description/urdf/xarm5/xarm5_robot_macro.xacro (robot description, xacro)
@@ -13,5 +13,5 @@
     baud_checkset:=true
     default_gripper_baud:=2000000
-    model1300:=false
+    model_num:=0
     inertial_params_filename:=''
     kinematics_params_filename:=''
@@ -45,5 +45,5 @@
         joint4_lower_limit="${-1.69297}" joint4_upper_limit="${pi*0.99}"
         joint5_lower_limit="${-pi*0.99}" joint5_upper_limit="${pi*0.99}"
-        model1300="${model1300}"
+        model_num="${model_num}"
         inertial_params_filename="${inertial_params_filename}"
         kinematics_params_filename="${kinematics_params_filename}"
@@ -58,5 +58,5 @@
           baud_checkset="${baud_checkset}" default_gripper_baud="${default_gripper_baud}" />
       </xacro:if>
-      <xacro:xarm5_urdf prefix="${prefix}" model1300="${model1300}"
+      <xacro:xarm5_urdf prefix="${prefix}" model_num="${model_num}"
         inertial_params_filename="${inertial_params_filename}"
         kinematics_params_filename="${kinematics_params_filename}"

File: xarm_ros2/xarm_description/urdf/xarm6/xarm6.urdf.xacro (robot description, xacro)
@@ -8,15 +8,27 @@
     joint5_lower_limit:=${-1.69297}  joint5_upper_limit:=${pi}
     joint6_lower_limit:=${-2.0*pi}  joint6_upper_limit:=${2.0*pi}
-    model1300:=false
+    model_num:=0
     inertial_params_filename:='' kinematics_params_filename:='' "
     >
     <!-- define property -->
-    <xacro:if value="${model1300}">
-      <xacro:property name="end_tool_visual_filename" value="end_tool/visual/end_tool_1300"/>
-      <xacro:property name="end_tool_collision_filename" value="end_tool/collision/end_tool_1300"/>
+    <xacro:if value="${model_num >= 1305 and model_num != 1380}">
+      <xacro:property name="model_dir" value="xarm6_1305"/>
+      <xacro:property name="link5_visual" value="xarm6_1305/visual/link5"/>
+      <xacro:property name="link5_collision" value="xarm6_1305/collision/link5"/>
+      <xacro:property name="link6_visual" value="xarm6_1305/visual/link6"/>
+      <xacro:property name="link6_collision" value="xarm6_1305/visual/link6"/>
     </xacro:if>
-    <xacro:unless value="${model1300}">
-      <xacro:property name="end_tool_visual_filename" value="xarm6/visual/link6"/>
-      <xacro:property name="end_tool_collision_filename" value="end_tool/collision/end_tool"/>
+    <xacro:unless value="${model_num >= 1305 and model_num != 1380}">
+      <xacro:property name="model_dir" value="xarm6"/>
+      <xacro:property name="link5_visual" value="xarm6/visual/link5"/>
+      <xacro:property name="link5_collision" value="xarm6/visual/link5"/>
+      <xacro:if value="${model_num >= 1300}">
+        <xacro:property name="link6_visual" value="end_tool/visual/end_tool_1300"/>
+        <xacro:property name="link6_collision" value="end_tool/collision/end_tool_1300"/>
+      </xacro:if>
+      <xacro:unless value="${model_num >= 1300}">
+        <xacro:property name="link6_visual" value="xarm6/visual/link6"/>
+        <xacro:property name="link6_collision" value="end_tool/collision/end_tool"/>
+      </xacro:unless>
     </xacro:unless>
     <!-- load params and define property -->
@@ -46,10 +58,10 @@
       </inertial>
       <xacro:common_link_visual
-        mesh_filename="xarm6/visual/link_base"
-        origin_xyz="0 0 0"
-        origin_rpy="0 0 0"
-        material_name="${prefix}White" />
-      <xacro:common_link_collision
-        mesh_filename="xarm6/visual/link_base"
+        mesh_filename="${model_dir}/visual/link_base"
+        origin_xyz="0 0 0"
+        origin_rpy="0 0 0"
+        material_name="${prefix}White" />
+      <xacro:common_link_collision
+        mesh_filename="${model_dir}/visual/link_base"
         origin_xyz="0 0 0"
         origin_rpy="0 0 0" />
@@ -60,10 +72,10 @@
         origin_rpy="0 0 0"/>
       <xacro:common_link_visual
-        mesh_filename="xarm6/visual/link1"
-        origin_xyz="0 0 0"
-        origin_rpy="0 0 0"
-        material_name="${prefix}White" />
-      <xacro:common_link_collision
-        mesh_filename="xarm6/visual/link1"
+        mesh_filename="${model_dir}/visual/link1"
+        origin_xyz="0 0 0"
+        origin_rpy="0 0 0"
+        material_name="${prefix}White" />
+      <xacro:common_link_collision
+        mesh_filename="${model_dir}/visual/link1"
         origin_xyz="0 0 0"
         origin_rpy="0 0 0" />
@@ -87,10 +99,10 @@
         origin_rpy="0 0 0"/>
       <xacro:common_link_visual
-        mesh_filename="xarm6/visual/link2"
+        mesh_filename="${model_dir}/visual/link2"
         origin_xyz="0 0 ${-kinematics_params['joint2']['y']}"
         origin_rpy="0 0 0"
         material_name="${prefix}White" />
       <xacro:common_link_collision
-        mesh_filename="xarm6/visual/link2"
+        mesh_filename="${model_dir}/visual/link2"
         origin_xyz="0 0 ${-kinematics_params['joint2']['y']}"
         origin_rpy="0 0 0" />
@@ -114,10 +126,10 @@
         origin_rpy="0 0 0"/>
       <xacro:common_link_visual
-        mesh_filename="xarm6/visual/link3"
-        origin_xyz="0 0 0"
-        origin_rpy="0 0 0"
-        material_name="${prefix}White" />
-      <xacro:common_link_collision
-        mesh_filename="xarm6/visual/link3"
+        mesh_filename="${model_dir}/visual/link3"
+        origin_xyz="0 0 0"
+        origin_rpy="0 0 0"
+        material_name="${prefix}White" />
+      <xacro:common_link_collision
+        mesh_filename="${model_dir}/visual/link3"
         origin_xyz="0 0 0"
         origin_rpy="0 0 0" />
@@ -141,10 +153,10 @@
         origin_rpy="0 0 0"/>
       <xacro:common_link_visual
-        mesh_filename="xarm6/visual/link4"
-        origin_xyz="0 0 0"
-        origin_rpy="0 0 0"
-        material_name="${prefix}White" />
-      <xacro:common_link_collision
-        mesh_filename="xarm6/visual/link4"
+        mesh_filename="${model_dir}/visual/link4"
+        origin_xyz="0 0 0"
+        origin_rpy="0 0 0"
+        material_name="${prefix}White" />
+      <xacro:common_link_collision
+        mesh_filename="${model_dir}/visual/link4"
         origin_xyz="0 0 0"
         origin_rpy="0 0 0" />
@@ -168,10 +180,10 @@
         origin_rpy="0 0 0"/>
       <xacro:common_link_visual
-        mesh_filename="xarm6/visual/link5"
-        origin_xyz="0 0 0"
-        origin_rpy="0 0 0"
-        material_name="${prefix}White" />
-      <xacro:common_link_collision
-        mesh_filename="xarm6/visual/link5"
+        mesh_filename="${link5_visual}"
+        origin_xyz="0 0 0"
+        origin_rpy="0 0 0"
+        material_name="${prefix}White" />
+      <xacro:common_link_collision
+        mesh_filename="${link5_collision}"
         origin_xyz="0 0 0"
         origin_rpy="0 0 0" />
@@ -194,10 +206,10 @@
         origin_rpy="0 0 0"/>
       <xacro:common_link_visual
-        mesh_filename="${end_tool_visual_filename}"
+        mesh_filename="${link6_visual}"
         origin_xyz="0 0 0"
         origin_rpy="0 0 0"
         material_name="${prefix}Silver" />
       <xacro:common_link_collision
-        mesh_filename="${end_tool_collision_filename}"
+        mesh_filename="${link6_collision}"
         origin_xyz="0 0 0"
         origin_rpy="0 0 0" />
