Commit message: Updated xarm ros2 ws with init compatibility test

File: xarm_ros2/xarm_description/urdf/xarm6/xarm6_robot_macro.xacro (robot description, xacro)
@@ -13,5 +13,5 @@
     baud_checkset:='true'
     default_gripper_baud:=2000000
-    model1300:=false
+    model_num:=0
     inertial_params_filename:=''
     kinematics_params_filename:=''
@@ -47,5 +47,5 @@
         joint5_lower_limit="${-1.69297}" joint5_upper_limit="${pi*0.99}"
         joint6_lower_limit="${-pi*0.99}" joint6_upper_limit="${pi*0.99}"
-        model1300="${model1300}"
+        model_num="${model_num}"
         inertial_params_filename="${inertial_params_filename}"
         kinematics_params_filename="${kinematics_params_filename}"
@@ -60,5 +60,5 @@
           baud_checkset="${baud_checkset}" default_gripper_baud="${default_gripper_baud}" />
       </xacro:if>
-      <xacro:xarm6_urdf prefix="${prefix}" model1300="${model1300}"
+      <xacro:xarm6_urdf prefix="${prefix}" model_num="${model_num}"
         inertial_params_filename="${inertial_params_filename}"
         kinematics_params_filename="${kinematics_params_filename}"

File: xarm_ros2/xarm_description/urdf/xarm7/xarm7.urdf.xacro (robot description, xacro)
@@ -9,15 +9,15 @@
     joint6_lower_limit:=${-1.69297}  joint6_upper_limit:=${pi}
     joint7_lower_limit:=${-2.0*pi}  joint7_upper_limit:=${2.0*pi}
-    model1300:=false
+    model_num:=0
     inertial_params_filename:='' kinematics_params_filename:='' "
     >
     <!-- define property -->
-    <xacro:if value="${model1300}">
-      <xacro:property name="end_tool_visual_filename" value="end_tool/visual/end_tool_1300"/>
-      <xacro:property name="end_tool_collision_filename" value="end_tool/collision/end_tool_1300"/>
+    <xacro:if value="${model_num >= 1300}">
+      <xacro:property name="link7_visual" value="end_tool/visual/end_tool_1300"/>
+      <xacro:property name="link7_collision" value="end_tool/collision/end_tool_1300"/>
     </xacro:if>
-    <xacro:unless value="${model1300}">
-      <xacro:property name="end_tool_visual_filename" value="xarm7/visual/link7"/>
-      <xacro:property name="end_tool_collision_filename" value="end_tool/collision/end_tool"/>
+    <xacro:unless value="${model_num >= 1300}">
+      <xacro:property name="link7_visual" value="xarm7/visual/link7"/>
+      <xacro:property name="link7_collision" value="end_tool/collision/end_tool"/>
     </xacro:unless>
     <!-- load params and define property -->
@@ -223,10 +223,10 @@
         origin_rpy="0 0 0"/>
       <xacro:common_link_visual
-        mesh_filename="${end_tool_visual_filename}"
+        mesh_filename="${link7_visual}"
         origin_xyz="0 0 0"
         origin_rpy="0 0 0"
         material_name="${prefix}Silver" />
       <xacro:common_link_collision
-        mesh_filename="${end_tool_collision_filename}"
+        mesh_filename="${link7_collision}"
         origin_xyz="0 0 0"
         origin_rpy="0 0 0" />

File: xarm_ros2/xarm_description/urdf/xarm7/xarm7_robot_macro.xacro (robot description, xacro)
@@ -13,5 +13,5 @@
     baud_checkset:='true'
     default_gripper_baud:=2000000
-    model1300:=false
+    model_num:=0
     inertial_params_filename:=''
     kinematics_params_filename:=''
@@ -49,5 +49,5 @@
         joint6_lower_limit="${-1.75}" joint6_upper_limit="${pi*0.99}"
         joint7_lower_limit="${-pi*0.99}" joint7_upper_limit="${pi*0.99}"
-        model1300="${model1300}"
+        model_num="${model_num}"
         inertial_params_filename="${inertial_params_filename}"
         kinematics_params_filename="${kinematics_params_filename}"
@@ -62,5 +62,5 @@
           baud_checkset="${baud_checkset}" default_gripper_baud="${default_gripper_baud}" />
       </xacro:if>
-      <xacro:xarm7_urdf prefix="${prefix}" model1300="${model1300}"
+      <xacro:xarm7_urdf prefix="${prefix}" model_num="${model_num}"
         inertial_params_filename="${inertial_params_filename}"
         kinematics_params_filename="${kinematics_params_filename}"

File: xarm_ros2/xarm_description/urdf/xarm7_mirror/xarm7_mirror.urdf.xacro (robot description, xacro)
@@ -9,5 +9,5 @@
     joint6_lower_limit:=${-pi}      joint6_upper_limit:=${1.69297}
     joint7_lower_limit:=${-2.0*pi}  joint7_upper_limit:=${2.0*pi}
-    model1300:=false
+    model_num:=0
     inertial_params_filename:='' kinematics_params_filename:='' "
     >

File: xarm_ros2/xarm_description/urdf/xarm7_mirror/xarm7_mirror_robot_macro.xacro (robot description, xacro)
@@ -13,5 +13,5 @@
     baud_checkset:='true'
     default_gripper_baud:=2000000
-    model1300:=false
+    model_num:=0
     inertial_params_filename:=''
     kinematics_params_filename:=''
@@ -49,5 +49,5 @@
         joint6_lower_limit="${-pi*0.99}" joint6_upper_limit="${1.75}"
         joint7_lower_limit="${-pi*0.99}" joint7_upper_limit="${pi*0.99}"
-        model1300="${model1300}"
+        model_num="${model_num}"
         inertial_params_filename="${inertial_params_filename}"
         kinematics_params_filename="${kinematics_params_filename}"
@@ -62,5 +62,5 @@
           baud_checkset="${baud_checkset}" default_gripper_baud="${default_gripper_baud}" />
       </xacro:if>
-      <xacro:xarm7_mirror_urdf prefix="${prefix}" model1300="${model1300}"
+      <xacro:xarm7_mirror_urdf prefix="${prefix}" model_num="${model_num}"
         inertial_params_filename="${inertial_params_filename}"
         kinematics_params_filename="${kinematics_params_filename}"

File: xarm_ros2/xarm_description/urdf/xarm_device_macro.xacro (robot description, xacro)
@@ -63,5 +63,5 @@
     <xacro:parse_link_inertial_filename dof="${dof}" robot_type="${robot_type}" robot_sn="${robot_sn}" model1300="${model1300}" />
     <xacro:property name="inertial_params_filename" value="${scope_parent_inertial_params_filename}"/>
-    <xacro:property name="new_model1300" value="${scope_parent_model1300}"/>
+    <xacro:property name="model_num" value="${scope_parent_model_num}"/>
     <!-- add one world link if no 'attach_to' specified  -->
     <xacro:if value="${attach_to == 'world' and create_attach_link}">
@@ -108,5 +108,5 @@
         baud_checkset="${baud_checkset}"
         default_gripper_baud="${default_gripper_baud}"
-        model1300="${new_model1300}"
+        model_num="${model_num}"
         inertial_params_filename="${inertial_params_filename}"
         kinematics_params_filename="${kinematics_params_filename}"
@@ -126,5 +126,5 @@
           baud_checkset="${baud_checkset}"
           default_gripper_baud="${default_gripper_baud}"
-          model1300="${new_model1300}"
+          model_num="${model_num}"
           inertial_params_filename="${inertial_params_filename}"
           kinematics_params_filename="${kinematics_params_filename}"
@@ -142,4 +142,5 @@
           baud_checkset="${baud_checkset}"
           default_gripper_baud="${default_gripper_baud}"
+          model_num="${model_num}"
           inertial_params_filename="${inertial_params_filename}"
           kinematics_params_filename="${kinematics_params_filename}"
@@ -158,5 +159,5 @@
           baud_checkset="${baud_checkset}"
           default_gripper_baud="${default_gripper_baud}"
-          model1300="${new_model1300}"
+          model_num="${model_num}"
           inertial_params_filename="${inertial_params_filename}"
           kinematics_params_filename="${kinematics_params_filename}"
@@ -177,5 +178,5 @@
           baud_checkset="${baud_checkset}"
           default_gripper_baud="${default_gripper_baud}"
-          model1300="${new_model1300}"
+          model_num="${model_num}"
           inertial_params_filename="${inertial_params_filename}"
           kinematics_params_filename="${kinematics_params_filename}"
@@ -194,5 +195,5 @@
           baud_checkset="${baud_checkset}"
           default_gripper_baud="${default_gripper_baud}"
-          model1300="${new_model1300}"
+          model_num="${model_num}"
           inertial_params_filename="${inertial_params_filename}"
           kinematics_params_filename="${kinematics_params_filename}"

File: xarm_ros2/xarm_moveit_config/srdf/xarm.srdf.xacro (robot description, xacro)
@@ -3,5 +3,5 @@
   <!-- parameters -->
   <xacro:arg name="prefix" default="" />
-  <xacro:arg name="dof" default="6" />
+  <xacro:arg name="dof" default="7" />
   <xacro:arg name="robot_type" default="xarm" />
   <xacro:arg name="add_gripper" default="false"/>
