Commit message: Refreshed xarm and depthai repos- still needs testing

File: xarm_ros2/xarm_description/urdf/common/common.link.xacro (robot description, xacro)
@@ -24,5 +24,5 @@
     </xacro:unless>
   </xacro:macro>
-  <xacro:macro name="common_link_visual" params="mesh_filename add_mesh_suffix:=true material_name:='White' origin_xyz:='0 0 0' origin_rpy:='0 0 0'">
+  <xacro:macro name="common_link_visual" params="mesh_filename add_mesh_suffix:=true material_name:='White' origin_xyz:='0 0 0' origin_rpy:='0 0 0' other_mesh_suffix:=''">
     <visual>
       <geometry>
@@ -31,5 +31,10 @@
         </xacro:if>
         <xacro:unless value="${add_mesh_suffix}">
-          <mesh filename="${mesh_path}/${mesh_filename}"/>
+          <xacro:if value="${other_mesh_suffix != ''}">
+            <mesh filename="${mesh_path}/${mesh_filename}.${other_mesh_suffix}"/>
+          </xacro:if>
+          <xacro:unless value="${other_mesh_suffix != ''}">
+            <mesh filename="${mesh_path}/${mesh_filename}"/>
+          </xacro:unless>
         </xacro:unless>
       </geometry>
@@ -38,5 +43,5 @@
     </visual>
   </xacro:macro>
-  <xacro:macro name="common_link_collision" params="mesh_filename add_mesh_suffix:=true origin_xyz:='0 0 0' origin_rpy:='0 0 0'">
+  <xacro:macro name="common_link_collision" params="mesh_filename add_mesh_suffix:=true origin_xyz:='0 0 0' origin_rpy:='0 0 0' other_mesh_suffix:=''">
     <collision>
       <geometry>
@@ -45,5 +50,10 @@
         </xacro:if>
         <xacro:unless value="${add_mesh_suffix}">
-          <mesh filename="${mesh_path}/${mesh_filename}"/>
+          <xacro:if value="${other_mesh_suffix != ''}">
+            <mesh filename="${mesh_path}/${mesh_filename}.${other_mesh_suffix}"/>
+          </xacro:if>
+          <xacro:unless value="${other_mesh_suffix != ''}">
+            <mesh filename="${mesh_path}/${mesh_filename}"/>
+          </xacro:unless>
         </xacro:unless>
       </geometry>
@@ -124,8 +134,8 @@
       </xacro:unless>
       <xacro:property name="date_int" value="${int(date_str)}" />
-      <xacro:if value="${robot_sn[11] == 'B' or robot_sn[11] == 'L' or robot_sn[11] == 'X' or robot_sn[11] == 'D'}">
+      <xacro:if value="${robot_sn[11] == 'B' or robot_sn[11] == 'L' or robot_sn[11] == 'X' or robot_sn[11] == 'D' or robot_sn[11] == 'A'}">
         <xacro:property name="hd_type" value="${robot_sn[11]}" />
       </xacro:if>
-      <xacro:unless value="${robot_sn[11] == 'B' or robot_sn[11] == 'L' or robot_sn[11] == 'X' or robot_sn[11] == 'D'}">
+      <xacro:unless value="${robot_sn[11] == 'B' or robot_sn[11] == 'L' or robot_sn[11] == 'X' or robot_sn[11] == 'D' or robot_sn[11] == 'A'}">
         <xacro:if value="${robot_sn_len >= 16 and robot_sn[14] == '_'}">
           <xacro:property name="hd_type" value="${robot_sn[15]}" />
@@ -164,4 +174,7 @@
             <xacro:property name="inertial_params_filename" value="xarm5_type5_HT_LD"/>
           </xacro:if>
+          <xacro:if value="${mass_type == 3}">
+            <xacro:property name="inertial_params_filename" value="xarm5_type5_UJ_BR_2403"/>
+          </xacro:if>
           <xacro:if value="${mass_type == 11}">
             <xacro:property name="inertial_params_filename" value="xarm5_type5_HT_BR2"/>
@@ -218,4 +231,7 @@
             <xacro:property name="inertial_params_filename" value="xarm7_type7_HT_LD"/>
           </xacro:if>
+          <xacro:if value="${mass_type == 3}">
+            <xacro:property name="inertial_params_filename" value="xarm7_type7_UJ_BR_2403"/>
+          </xacro:if>
           <xacro:if value="${mass_type == 11}">
             <xacro:property name="inertial_params_filename" value="xarm7_type7_HT_BR2"/>

File: xarm_ros2/xarm_description/urdf/gripper/bio_gripper.ros2_control.xacro (robot description, xacro)
@@ -3,5 +3,5 @@
   <xacro:macro name="bio_gripper_ros2_control" params="prefix:=''
     ros2_control_plugin:='uf_robot_hardware/UFRobotFakeSystemHardware' ">
-    <ros2_control name="BioGripperSystem" type="system">
+    <ros2_control name="${prefix}BioGripperSystem" type="system">
       <hardware>
         <plugin>${ros2_control_plugin}</plugin>

File: xarm_ros2/xarm_description/urdf/gripper/xarm_gripper.ros2_control.xacro (robot description, xacro)
@@ -3,5 +3,5 @@
   <xacro:macro name="xarm_gripper_ros2_control" params="prefix:=''
     ros2_control_plugin:='uf_robot_hardware/UFRobotFakeSystemHardware' ">
-    <ros2_control name="XArmGripperSystem" type="system">
+    <ros2_control name="${prefix}XArmGripperSystem" type="system">
       <hardware>
         <plugin>${ros2_control_plugin}</plugin>

File: xarm_ros2/xarm_description/urdf/xarm5/xarm5.urdf.xacro (robot description, xacro)
@@ -11,11 +11,25 @@
     >
     <!-- define property -->
-    <xacro:if value="${model_num >= 1300}">
-      <xacro:property name="link5_visual" value="end_tool/visual/end_tool_1300"/>
-      <xacro:property name="link5_collision" value="end_tool/collision/end_tool_1300"/>
+    <xacro:if value="${model_num >= 1305 and model_num != 1380}">
+      <xacro:property name="visual_dir" value="xarm5_1305/visual"/>
+      <xacro:property name="collision_dir" value="xarm5_1305/collision"/>
+      <xacro:property name="add_mesh_suffix" value="false"/>
+      <xacro:property name="collison_mesh_suffix" value="obj"/>
+      <xacro:property name="link5_visual" value="xarm5_1305/visual/link5"/>
+      <xacro:property name="link5_collision" value="xarm5_1305/collision/link5"/>
     </xacro:if>
-    <xacro:unless value="${model_num >= 1300}">
-      <xacro:property name="link5_visual" value="xarm5/visual/link5"/>
-      <xacro:property name="link5_collision" value="end_tool/collision/end_tool"/>
+    <xacro:unless value="${model_num >= 1305 and model_num != 1380}">
+      <xacro:property name="visual_dir" value="xarm5/visual"/>
+      <xacro:property name="collision_dir" value="xarm5/visual"/>
+      <xacro:property name="add_mesh_suffix" value="true"/>
+      <xacro:property name="collison_mesh_suffix" value="stl"/>
+      <xacro:if value="${model_num >= 1300}">
+        <xacro:property name="link5_visual" value="end_tool/visual/end_tool_1300"/>
+        <xacro:property name="link5_collision" value="end_tool/collision/end_tool_1300"/>
+      </xacro:if>
+      <xacro:unless value="${model_num >= 1300}">
+        <xacro:property name="link5_visual" value="xarm5/visual/link5"/>
+        <xacro:property name="link5_collision" value="end_tool/collision/end_tool"/>
+      </xacro:unless>
     </xacro:unless>
     <!-- load params and define property -->
@@ -45,10 +59,12 @@
       </inertial>
       <xacro:common_link_visual
-        mesh_filename="xarm5/visual/link_base"
-        origin_xyz="0 0 0"
-        origin_rpy="0 0 0"
-        material_name="${prefix}White" />
-      <xacro:common_link_collision
-        mesh_filename="xarm5/visual/link_base"
+        mesh_filename="${visual_dir}/link_base"
+        origin_xyz="0 0 0"
+        origin_rpy="0 0 0"
+        material_name="${prefix}White" />
+      <xacro:common_link_collision
+        mesh_filename="${collision_dir}/link_base"
+        add_mesh_suffix="${add_mesh_suffix}"
+        other_mesh_suffix="${collison_mesh_suffix}"
         origin_xyz="0 0 0"
         origin_rpy="0 0 0" />
@@ -59,10 +75,12 @@
         origin_rpy="0 0 0"/>
       <xacro:common_link_visual
-        mesh_filename="xarm5/visual/link1"
-        origin_xyz="0 0 0"
-        origin_rpy="0 0 0"
-        material_name="${prefix}White" />
-      <xacro:common_link_collision
-        mesh_filename="xarm5/visual/link1"
+        mesh_filename="${visual_dir}/link1"
+        origin_xyz="0 0 0"
+        origin_rpy="0 0 0"
+        material_name="${prefix}White" />
+      <xacro:common_link_collision
+        mesh_filename="${collision_dir}/link1"
+        add_mesh_suffix="${add_mesh_suffix}"
+        other_mesh_suffix="${collison_mesh_suffix}"
         origin_xyz="0 0 0"
         origin_rpy="0 0 0" />
@@ -86,10 +104,12 @@
         origin_rpy="0 0 0"/>
       <xacro:common_link_visual
-        mesh_filename="xarm5/visual/link2"
-        origin_xyz="0 0 0"
-        origin_rpy="0 0 0"
-        material_name="${prefix}White" />
-      <xacro:common_link_collision
-        mesh_filename="xarm5/visual/link2"
+        mesh_filename="${visual_dir}/link2"
+        origin_xyz="0 0 0"
+        origin_rpy="0 0 0"
+        material_name="${prefix}White" />
+      <xacro:common_link_collision
+        mesh_filename="${collision_dir}/link2"
+        add_mesh_suffix="${add_mesh_suffix}"
+        other_mesh_suffix="${collison_mesh_suffix}"
         origin_xyz="0 0 0"
         origin_rpy="0 0 0" />
@@ -113,10 +133,12 @@
         origin_rpy="0 0 0"/>
       <xacro:common_link_visual
-        mesh_filename="xarm5/visual/link3"
-        origin_xyz="0 0 0"
-        origin_rpy="0 0 0"
-        material_name="${prefix}White" />
-      <xacro:common_link_collision
-        mesh_filename="xarm5/visual/link3"
+        mesh_filename="${visual_dir}/link3"
+        origin_xyz="0 0 0"
+        origin_rpy="0 0 0"
+        material_name="${prefix}White" />
+      <xacro:common_link_collision
+        mesh_filename="${collision_dir}/link3"
+        add_mesh_suffix="${add_mesh_suffix}"
+        other_mesh_suffix="${collison_mesh_suffix}"
         origin_xyz="0 0 0"
         origin_rpy="0 0 0" />
@@ -140,10 +162,12 @@
         origin_rpy="0 0 0"/>
       <xacro:common_link_visual
-        mesh_filename="xarm5/visual/link4"
-        origin_xyz="0 0 0"
-        origin_rpy="0 0 0"
-        material_name="${prefix}White" />
-      <xacro:common_link_collision
-        mesh_filename="xarm5/visual/link4"
+        mesh_filename="${visual_dir}/link4"
+        origin_xyz="0 0 0"
+        origin_rpy="0 0 0"
+        material_name="${prefix}White" />
+      <xacro:common_link_collision
+        mesh_filename="${collision_dir}/link4"
+        add_mesh_suffix="${add_mesh_suffix}"
+        other_mesh_suffix="${collison_mesh_suffix}"
         origin_xyz="0 0 0"
         origin_rpy="0 0 0" />
@@ -173,4 +197,6 @@
       <xacro:common_link_collision
         mesh_filename="${link5_collision}"
+        add_mesh_suffix="${add_mesh_suffix}"
+        other_mesh_suffix="${collison_mesh_suffix}"
         origin_xyz="0 0 0"
         origin_rpy="0 0 0" />

File: xarm_ros2/xarm_description/urdf/xarm6/xarm6.urdf.xacro (robot description, xacro)
@@ -13,14 +13,16 @@
     <!-- define property -->
     <xacro:if value="${model_num >= 1305 and model_num != 1380}">
-      <xacro:property name="model_dir" value="xarm6_1305"/>
-      <xacro:property name="link5_visual" value="xarm6_1305/visual/link5"/>
-      <xacro:property name="link5_collision" value="xarm6_1305/collision/link5"/>
+      <xacro:property name="visual_dir" value="xarm6_1305/visual"/>
+      <xacro:property name="collision_dir" value="xarm6_1305/collision"/>
+      <xacro:property name="add_mesh_suffix" value="false"/>
+      <xacro:property name="collison_mesh_suffix" value="obj"/>
       <xacro:property name="link6_visual" value="xarm6_1305/visual/link6"/>
-      <xacro:property name="link6_collision" value="xarm6_1305/visual/link6"/>
+      <xacro:property name="link6_collision" value="xarm6_1305/collision/link6"/>
     </xacro:if>
     <xacro:unless value="${model_num >= 1305 and model_num != 1380}">
-      <xacro:property name="model_dir" value="xarm6"/>
-      <xacro:property name="link5_visual" value="xarm6/visual/link5"/>
-      <xacro:property name="link5_collision" value="xarm6/visual/link5"/>
+      <xacro:property name="visual_dir" value="xarm6/visual"/>
+      <xacro:property name="collision_dir" value="xarm6/visual"/>
+      <xacro:property name="add_mesh_suffix" value="true"/>
+      <xacro:property name="collison_mesh_suffix" value="stl"/>
       <xacro:if value="${model_num >= 1300}">
         <xacro:property name="link6_visual" value="end_tool/visual/end_tool_1300"/>
@@ -58,10 +60,12 @@
       </inertial>
       <xacro:common_link_visual
-        mesh_filename="${model_dir}/visual/link_base"
-        origin_xyz="0 0 0"
-        origin_rpy="0 0 0"
-        material_name="${prefix}White" />
-      <xacro:common_link_collision
-        mesh_filename="${model_dir}/visual/link_base"
+        mesh_filename="${visual_dir}/link_base"
+        origin_xyz="0 0 0"
+        origin_rpy="0 0 0"
+        material_name="${prefix}White" />
+      <xacro:common_link_collision
+        mesh_filename="${collision_dir}/link_base"
+        add_mesh_suffix="${add_mesh_suffix}"
+        other_mesh_suffix="${collison_mesh_suffix}"
         origin_xyz="0 0 0"
         origin_rpy="0 0 0" />
@@ -72,10 +76,12 @@
         origin_rpy="0 0 0"/>
       <xacro:common_link_visual
-        mesh_filename="${model_dir}/visual/link1"
-        origin_xyz="0 0 0"
-        origin_rpy="0 0 0"
-        material_name="${prefix}White" />
-      <xacro:common_link_collision
-        mesh_filename="${model_dir}/visual/link1"
+        mesh_filename="${visual_dir}/link1"
+        origin_xyz="0 0 0"
+        origin_rpy="0 0 0"
+        material_name="${prefix}White" />
+      <xacro:common_link_collision
+        mesh_filename="${collision_dir}/link1"
+        add_mesh_suffix="${add_mesh_suffix}"
+        other_mesh_suffix="${collison_mesh_suffix}"
         origin_xyz="0 0 0"
         origin_rpy="0 0 0" />
@@ -99,11 +105,13 @@
         origin_rpy="0 0 0"/>
       <xacro:common_link_visual
-        mesh_filename="${model_dir}/visual/link2"
-        origin_xyz="0 0 ${-kinematics_params['joint2']['y']}"
-        origin_rpy="0 0 0"
-        material_name="${prefix}White" />
-      <xacro:common_link_collision
-        mesh_filename="${model_dir}/visual/link2"
-        origin_xyz="0 0 ${-kinematics_params['joint2']['y']}"
+        mesh_filename="${visual_dir}/link2"
+        origin_xyz="0 0 0"
+        origin_rpy="0 0 0"
+        material_name="${prefix}White" />
+      <xacro:common_link_collision
+        mesh_filename="${collision_dir}/link2"
+        add_mesh_suffix="${add_mesh_suffix}"
+        other_mesh_suffix="${collison_mesh_suffix}"
+        origin_xyz="0 0 0"
         origin_rpy="0 0 0" />
     </link>
@@ -126,10 +134,12 @@
         origin_rpy="0 0 0"/>
       <xacro:common_link_visual
-        mesh_filename="${model_dir}/visual/link3"
-        origin_xyz="0 0 0"
-        origin_rpy="0 0 0"
-        material_name="${prefix}White" />
-      <xacro:common_link_collision
-        mesh_filename="${model_dir}/visual/link3"
+        mesh_filename="${visual_dir}/link3"
+        origin_xyz="0 0 0"
+        origin_rpy="0 0 0"
+        material_name="${prefix}White" />
+      <xacro:common_link_collision
+        mesh_filename="${collision_dir}/link3"
+        add_mesh_suffix="${add_mesh_suffix}"
+        other_mesh_suffix="${collison_mesh_suffix}"
         origin_xyz="0 0 0"
         origin_rpy="0 0 0" />
@@ -153,10 +163,12 @@
         origin_rpy="0 0 0"/>
       <xacro:common_link_visual
-        mesh_filename="${model_dir}/visual/link4"
-        origin_xyz="0 0 0"
-        origin_rpy="0 0 0"
-        material_name="${prefix}White" />
-      <xacro:common_link_collision
-        mesh_filename="${model_dir}/visual/link4"
+        mesh_filename="${visual_dir}/link4"
+        origin_xyz="0 0 0"
+        origin_rpy="0 0 0"
+        material_name="${prefix}White" />
+      <xacro:common_link_collision
+        mesh_filename="${collision_dir}/link4"
+        add_mesh_suffix="${add_mesh_suffix}"
+        other_mesh_suffix="${collison_mesh_suffix}"
         origin_xyz="0 0 0"
         origin_rpy="0 0 0" />
@@ -180,10 +192,12 @@
         origin_rpy="0 0 0"/>
       <xacro:common_link_visual
-        mesh_filename="${link5_visual}"
-        origin_xyz="0 0 0"
-        origin_rpy="0 0 0"
-        material_name="${prefix}White" />
-      <xacro:common_link_collision
-        mesh_filename="${link5_collision}"
+        mesh_filename="${visual_dir}/link5"
+        origin_xyz="0 0 0"
+        origin_rpy="0 0 0"
+        material_name="${prefix}White" />
+      <xacro:common_link_collision
+        mesh_filename="${collision_dir}/link5"
+        add_mesh_suffix="${add_mesh_suffix}"
+        other_mesh_suffix="${collison_mesh_suffix}"
         origin_xyz="0 0 0"
         origin_rpy="0 0 0" />
@@ -212,4 +226,6 @@
       <xacro:common_link_collision
         mesh_filename="${link6_collision}"
+        add_mesh_suffix="${add_mesh_suffix}"
+        other_mesh_suffix="${collison_mesh_suffix}"
         origin_xyz="0 0 0"
         origin_rpy="0 0 0" />
