Commit message: New urdf for testing

File: dim_cpp/urdf/alfred_base_descr.urdf (robot description, URDF)
Before this commit: robot alfred_base_descr, 8 links, 7 joints
Links:
- added link chest_cam_frame
- added link chest_cam_imu_frame
- added link chest_cam_left_camera_frame
- added link chest_cam_left_camera_optical_frame
- added link chest_cam_link
- added link chest_cam_model_origin; visual mesh filename=package://depthai_descriptions/urdf/models/OAK-D-PRO.stl
- added link chest_cam_rgb_camera_frame
- added link chest_cam_rgb_camera_optical_frame
- added link chest_cam_right_camera_frame
- added link chest_cam_right_camera_optical_frame
- added link head_cam_frame
- added link head_cam_imu_frame
- added link head_cam_left_camera_frame
- added link head_cam_left_camera_optical_frame
- added link head_cam_link
- added link head_cam_model_origin; visual mesh filename=package://depthai_descriptions/urdf/models/OAK-D-PRO.stl
- added link head_cam_rgb_camera_frame
- added link head_cam_rgb_camera_optical_frame
- added link head_cam_right_camera_frame
- added link head_cam_right_camera_optical_frame
- added link left_arm_mount
- added link leftleft_finger, mass 0.048304; collision mesh filename=package://xarm_description/meshes/gripper/xarm/left_finger.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; visual mesh filename=package://xarm_description/meshes/gripper/xarm/left_finger.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
- added link leftleft_inner_knuckle, mass 0.0230125781256706; collision mesh filename=package://xarm_description/meshes/gripper/xarm/left_inner_k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; visual mesh filename=package://xarm_description/meshes/gripper/xarm/left_inner_k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
- added link leftleft_outer_knuckle, mass 0.033618; collision mesh filename=package://xarm_description/meshes/gripper/xarm/left_outer_k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; visual mesh filename=package://xarm_description/meshes/gripper/xarm/left_outer_k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
- added link leftlink1, mass 2.3814; collision mesh filename=package://xarm_description/meshes/xarm6/visual/link1.stl; visual mesh filename=package://xarm_description/meshes/xarm6/visual/link1.stl
- added link leftlink2, mass 2.2675; collision mesh filename=package://xarm_description/meshes/xarm6/visual/link2.stl; visual mesh filename=package://xarm_description/meshes/xarm6/visual/link2.stl
- added link leftlink3, mass 1.875; collision mesh filename=package://xarm_description/meshes/xarm6/visual/link3.stl; visual mesh filename=package://xarm_description/meshes/xarm6/visual/link3.stl
- added link leftlink4, mass 1.3192; collision mesh filename=package://xarm_description/meshes/xarm6/visual/link4.stl; visual mesh filename=package://xarm_description/meshes/xarm6/visual/link4.stl
- added link leftlink5, mass 1.33854; collision mesh filename=package://xarm_description/meshes/xarm6/visual/link5.stl; visual mesh filename=package://xarm_description/meshes/xarm6/visual/link5.stl
- added link leftlink6, mass 0.17; collision mesh filename=package://xarm_description/meshes/end_tool/collision/end_to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; visual mesh filename=package://xarm_description/meshes/xarm6/visual/link6.stl
- added link leftlink_base, mass 2.7; collision mesh filename=package://xarm_description/meshes/xarm6/visual/link_base.stl; visual mesh filename=package://xarm_description/meshes/xarm6/visual/link_base.stl
- added link leftlink_eef
- added link leftlink_tcp
- added link leftright_finger, mass 0.048304; collision mesh filename=package://xarm_description/meshes/gripper/xarm/right_finger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; visual mesh filename=package://xarm_description/meshes/gripper/xarm/right_finger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
- added link leftright_inner_knuckle, mass 0.023013; collision mesh filename=package://xarm_description/meshes/gripper/xarm/right_inner_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; visual mesh filename=package://xarm_description/meshes/gripper/xarm/right_inner_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
- added link leftright_outer_knuckle, mass 0.033618; collision mesh filename=package://xarm_description/meshes/gripper/xarm/right_outer_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; visual mesh filename=package://xarm_description/meshes/gripper/xarm/right_outer_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
- added link leftxarm_gripper_base_link, mass 0.54156; collision mesh filename=package://xarm_description/meshes/gripper/xarm/base_link.stl; visual mesh filename=package://xarm_description/meshes/gripper/xarm/base_link.stl
- added link right_arm_mount
- added link rightleft_finger, mass 0.048304; collision mesh filename=package://xarm_description/meshes/gripper/xarm/left_finger.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; visual mesh filename=package://xarm_description/meshes/gripper/xarm/left_finger.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
- added link rightleft_inner_knuckle, mass 0.0230125781256706; collision mesh filename=package://xarm_description/meshes/gripper/xarm/left_inner_k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; visual mesh filename=package://xarm_description/meshes/gripper/xarm/left_inner_k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
- added link rightleft_outer_knuckle, mass 0.033618; collision mesh filename=package://xarm_description/meshes/gripper/xarm/left_outer_k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; visual mesh filename=package://xarm_description/meshes/gripper/xarm/left_outer_k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
- added link rightlink1, mass 2.382; collision mesh filename=package://xarm_description/meshes/xarm7/visual/link1.stl; visual mesh filename=package://xarm_description/meshes/xarm7/visual/link1.stl
- added link rightlink2, mass 1.869; collision mesh filename=package://xarm_description/meshes/xarm7/visual/link2.stl; visual mesh filename=package://xarm_description/meshes/xarm7/visual/link2.stl
- added link rightlink3, mass 1.6383; collision mesh filename=package://xarm_description/meshes/xarm7/visual/link3.stl; visual mesh filename=package://xarm_description/meshes/xarm7/visual/link3.stl
- added link rightlink4, mass 1.7269; collision mesh filename=package://xarm_description/meshes/xarm7/visual/link4.stl; visual mesh filename=package://xarm_description/meshes/xarm7/visual/link4.stl
- added link rightlink5, mass 1.3203; collision mesh filename=package://xarm_description/meshes/xarm7/visual/link5.stl; visual mesh filename=package://xarm_description/meshes/xarm7/visual/link5.stl
- added link rightlink6, mass 1.325; collision mesh filename=package://xarm_description/meshes/xarm7/visual/link6.stl; visual mesh filename=package://xarm_description/meshes/xarm7/visual/link6.stl
- added link rightlink7, mass 0.17; collision mesh filename=package://xarm_description/meshes/end_tool/collision/end_to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; visual mesh filename=package://xarm_description/meshes/xarm7/visual/link7.stl
- added link rightlink_base, mass 0.88556; collision mesh filename=package://xarm_description/meshes/xarm7/visual/link_base.stl; visual mesh filename=package://xarm_description/meshes/xarm7/visual/link_base.stl
- added link rightlink_eef
- added link rightlink_tcp
- added link rightright_finger, mass 0.048304; collision mesh filename=package://xarm_description/meshes/gripper/xarm/right_finger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; visual mesh filename=package://xarm_description/meshes/gripper/xarm/right_finger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
- added link rightright_inner_knuckle, mass 0.023013; collision mesh filename=package://xarm_description/meshes/gripper/xarm/right_inner_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; visual mesh filename=package://xarm_description/meshes/gripper/xarm/right_inner_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
- added link rightright_outer_knuckle, mass 0.033618; collision mesh filename=package://xarm_description/meshes/gripper/xarm/right_outer_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; visual mesh filename=package://xarm_description/meshes/gripper/xarm/right_outer_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
- added link rightxarm_gripper_base_link, mass 0.54156; collision mesh filename=package://xarm_description/meshes/gripper/xarm/base_link.stl; visual mesh filename=package://xarm_description/meshes/gripper/xarm/base_link.stl
Joints:
- added joint chest_cam_center_joint: type fixed, parent chest_cam_link, child chest_cam_frame, origin xyz=0 -0.022921 -0.004764 rpy=3.14159265 0 -1.5707963267948966
- added joint chest_cam_imu_joint: type fixed, parent chest_cam_frame, child chest_cam_imu_frame, origin xyz=-0.008 -0.037945 -0.00079 rpy=3.141592653589793 1.5707963267948966 0.0
- added joint chest_cam_joint: type fixed, parent alfred_base_link, child chest_cam_link, origin xyz=.225 -.455681 1.441731 rpy=0.78539816 0 0
- added joint chest_cam_left_camera_joint: type fixed, parent chest_cam_frame, child chest_cam_left_camera_frame, origin xyz=0 0.0375 0 rpy=0 0 0
- added joint chest_cam_left_camera_optical_joint: type fixed, parent chest_cam_left_camera_frame, child chest_cam_left_camera_optical_frame, origin xyz=0 0 0 rpy=-1.5707963267948966 0.0 -1.5707963267948966
- added joint chest_cam_model_origin_joint: type fixed, parent chest_cam_frame, child chest_cam_model_origin, origin xyz=0 0 0 rpy=1.5708 0 1.5708
- added joint chest_cam_rgb_camera_joint: type fixed, parent chest_cam_frame, child chest_cam_rgb_camera_frame, origin xyz=0 0 0 rpy=0 0 0
- added joint chest_cam_rgb_camera_optical_joint: type fixed, parent chest_cam_rgb_camera_frame, child chest_cam_rgb_camera_optical_frame, origin xyz=0 0 0 rpy=-1.5707963267948966 0.0 -1.5707963267948966
- added joint chest_cam_right_camera_joint: type fixed, parent chest_cam_frame, child chest_cam_right_camera_frame, origin xyz=0 -0.0375 0 rpy=0 0 0
- added joint chest_cam_right_camera_optical_joint: type fixed, parent chest_cam_right_camera_frame, child chest_cam_right_camera_optical_frame, origin xyz=0 0 0 rpy=-1.5707963267948966 0.0 -1.5707963267948966
- added joint head_cam_center_joint: type fixed, parent head_cam_link, child head_cam_frame, origin xyz=0 -0.022921 0.004764 rpy=0 0 -1.5707963267948966
- added joint head_cam_imu_joint: type fixed, parent head_cam_frame, child head_cam_imu_frame, origin xyz=-0.008 -0.037945 -0.00079 rpy=3.141592653589793 1.5707963267948966 0.0
- added joint head_cam_joint: type fixed, parent camera_holder, child head_cam_link, origin xyz=0 -0.0025 0.057 rpy=0 0 0
- added joint head_cam_left_camera_joint: type fixed, parent head_cam_frame, child head_cam_left_camera_frame, origin xyz=0 0.0375 0 rpy=0 0 0
- added joint head_cam_left_camera_optical_joint: type fixed, parent head_cam_left_camera_frame, child head_cam_left_camera_optical_frame, origin xyz=0 0 0 rpy=-1.5707963267948966 0.0 -1.5707963267948966
- added joint head_cam_model_origin_joint: type fixed, parent head_cam_frame, child head_cam_model_origin, origin xyz=0 0 0 rpy=1.5708 0 1.5708
- added joint head_cam_rgb_camera_joint: type fixed, parent head_cam_frame, child head_cam_rgb_camera_frame, origin xyz=0 0 0 rpy=0 0 0
- added joint head_cam_rgb_camera_optical_joint: type fixed, parent head_cam_rgb_camera_frame, child head_cam_rgb_camera_optical_frame, origin xyz=0 0 0 rpy=-1.5707963267948966 0.0 -1.5707963267948966
- added joint head_cam_right_camera_joint: type fixed, parent head_cam_frame, child head_cam_right_camera_frame, origin xyz=0 -0.0375 0 rpy=0 0 0
- added joint head_cam_right_camera_optical_joint: type fixed, parent head_cam_right_camera_frame, child head_cam_right_camera_optical_frame, origin xyz=0 0 0 rpy=-1.5707963267948966 0.0 -1.5707963267948966
- added joint left_arm_mount_joint: type fixed, parent pillar_platform, child left_arm_mount, origin xyz=.12325 -.319646 1.4125 rpy=1.57079633 0 -1.57079633
- added joint leftdrive_joint: type revolute, parent leftxarm_gripper_base_link, child leftleft_outer_knuckle, origin xyz=0 0.035 0.059098 rpy=0 0 0, axis 1 0 0, limit lower=0 upper=0.85 effort=50 velocity=2
- added joint leftgripper_fix: type fixed, parent leftlink_eef, child leftxarm_gripper_base_link, origin xyz=0 0 0 rpy=0 0 0
- added joint leftjoint1: type revolute, parent leftlink_base, child leftlink1, origin xyz=0 0 0.267 rpy=0 0 0, axis 0 0 1, limit lower=-6.283185307179586 upper=6.283185307179586 effort=50.0 velocity=3.14
- added joint leftjoint2: type revolute, parent leftlink1, child leftlink2, origin xyz=0 0 0 rpy=-1.5708 0 0, axis 0 0 1, limit lower=-2.059 upper=2.0944 effort=50.0 velocity=3.14
- added joint leftjoint3: type revolute, parent leftlink2, child leftlink3, origin xyz=0.0535 -0.2845 0 rpy=0 0 0, axis 0 0 1, limit lower=-3.927 upper=0.19198 effort=32.0 velocity=3.14
- added joint leftjoint4: type revolute, parent leftlink3, child leftlink4, origin xyz=0.0775 0.3425 0 rpy=-1.5708 0 0, axis 0 0 1, limit lower=-6.283185307179586 upper=6.283185307179586 effort=32.0 velocity=3.14
- added joint leftjoint5: type revolute, parent leftlink4, child leftlink5, origin xyz=0 0 0 rpy=1.5708 0 0, axis 0 0 1, limit lower=-1.69297 upper=3.141592653589793 effort=32.0 velocity=3.14
- added joint leftjoint6: type revolute, parent leftlink5, child leftlink6, origin xyz=0.076 0.097 0 rpy=-1.5708 0 0, axis 0 0 1, limit lower=-6.283185307179586 upper=6.283185307179586 effort=20.0 velocity=3.14
- added joint leftjoint_eef: type fixed, parent leftlink6, child leftlink_eef, origin xyz=0 0 0 rpy=0 0 0
- added joint leftjoint_tcp: type fixed, parent leftxarm_gripper_base_link, child leftlink_tcp, origin xyz=0 0 0.172 rpy=0 0 0
- added joint leftleft_finger_joint: type revolute, parent leftleft_outer_knuckle, child leftleft_finger, origin xyz=0 0.035465 0.042039 rpy=0 0 0, axis -1 0 0, limit lower=0 upper=0.85 effort=50 velocity=2, mimic joint=leftdrive_joint multiplier=1 offset=0
- added joint leftleft_inner_knuckle_joint: type revolute, parent leftxarm_gripper_base_link, child leftleft_inner_knuckle, origin xyz=0 0.02 0.074098 rpy=0 0 0, axis 1 0 0, limit lower=0 upper=0.85 effort=50 velocity=2, mimic joint=leftdrive_joint multiplier=1 offset=0
- added joint leftright_finger_joint: type revolute, parent leftright_outer_knuckle, child leftright_finger, origin xyz=0 -0.035465 0.042039 rpy=0 0 0, axis 1 0 0, limit lower=0 upper=0.85 effort=50 velocity=2, mimic joint=leftdrive_joint multiplier=1 offset=0
- added joint leftright_inner_knuckle_joint: type revolute, parent leftxarm_gripper_base_link, child leftright_inner_knuckle, origin xyz=0 -0.02 0.074098 rpy=0 0 0, axis -1 0 0, limit lower=0 upper=0.85 effort=50 velocity=2, mimic joint=leftdrive_joint multiplier=1 offset=0
- added joint leftright_outer_knuckle_joint: type revolute, parent leftxarm_gripper_base_link, child leftright_outer_knuckle, origin xyz=0 -0.035 0.059098 rpy=0 0 0, axis -1 0 0, limit lower=0 upper=0.85 effort=50 velocity=2, mimic joint=leftdrive_joint multiplier=1 offset=0
- added joint leftworld_joint: type fixed, parent left_arm_mount, child leftlink_base, origin xyz=0 0 0 rpy=0 0 0
- added joint right_arm_mount_joint: type fixed, parent pillar_platform, child right_arm_mount, origin xyz=.32675 -.319646 1.4125 rpy=1.57079633 3.14159265 1.57079633
- added joint rightdrive_joint: type revolute, parent rightxarm_gripper_base_link, child rightleft_outer_knuckle, origin xyz=0 0.035 0.059098 rpy=0 0 0, axis 1 0 0, limit lower=0 upper=0.85 effort=50 velocity=2
- added joint rightgripper_fix: type fixed, parent rightlink_eef, child rightxarm_gripper_base_link, origin xyz=0 0 0 rpy=0 0 0
- added joint rightjoint1: type revolute, parent rightlink_base, child rightlink1, origin xyz=0 0 0.267 rpy=0 0 0, axis 0 0 1, limit lower=-6.283185307179586 upper=6.283185307179586 effort=50 velocity=3.14
- added joint rightjoint2: type revolute, parent rightlink1, child rightlink2, origin xyz=0 0 0 rpy=-1.5708 0 0, axis 0 0 1, limit lower=-2.059 upper=2.0944 effort=50 velocity=3.14
- added joint rightjoint3: type revolute, parent rightlink2, child rightlink3, origin xyz=0 -0.293 0 rpy=1.5708 0 0, axis 0 0 1, limit lower=-6.283185307179586 upper=6.283185307179586 effort=30 velocity=3.14
- added joint rightjoint4: type revolute, parent rightlink3, child rightlink4, origin xyz=0.0525 0 0 rpy=1.5708 0 0, axis 0 0 1, limit lower=-0.19198 upper=3.927 effort=30 velocity=3.14
- added joint rightjoint5: type revolute, parent rightlink4, child rightlink5, origin xyz=0.0775 -0.3425 0 rpy=1.5708 0 0, axis 0 0 1, limit lower=-6.283185307179586 upper=6.283185307179586 effort=30 velocity=3.14
- added joint rightjoint6: type revolute, parent rightlink5, child rightlink6, origin xyz=0 0 0 rpy=1.5708 0 0, axis 0 0 1, limit lower=-1.69297 upper=3.141592653589793 effort=20 velocity=3.14
- added joint rightjoint7: type revolute, parent rightlink6, child rightlink7, origin xyz=0.076 0.097 0 rpy=-1.5708 0 0, axis 0 0 1, limit lower=-6.283185307179586 upper=6.283185307179586 effort=20 velocity=3.14
- added joint rightjoint_eef: type fixed, parent rightlink7, child rightlink_eef, origin xyz=0 0 0 rpy=0 0 0
- added joint rightjoint_tcp: type fixed, parent rightxarm_gripper_base_link, child rightlink_tcp, origin xyz=0 0 0.172 rpy=0 0 0
- added joint rightleft_finger_joint: type revolute, parent rightleft_outer_knuckle, child rightleft_finger, origin xyz=0 0.035465 0.042039 rpy=0 0 0, axis -1 0 0, limit lower=0 upper=0.85 effort=50 velocity=2, mimic joint=rightdrive_joint multiplier=1 offset=0
- added joint rightleft_inner_knuckle_joint: type revolute, parent rightxarm_gripper_base_link, child rightleft_inner_knuckle, origin xyz=0 0.02 0.074098 rpy=0 0 0, axis 1 0 0, limit lower=0 upper=0.85 effort=50 velocity=2, mimic joint=rightdrive_joint multiplier=1 offset=0
- added joint rightright_finger_joint: type revolute, parent rightright_outer_knuckle, child rightright_finger, origin xyz=0 -0.035465 0.042039 rpy=0 0 0, axis 1 0 0, limit lower=0 upper=0.85 effort=50 velocity=2, mimic joint=rightdrive_joint multiplier=1 offset=0
- added joint rightright_inner_knuckle_joint: type revolute, parent rightxarm_gripper_base_link, child rightright_inner_knuckle, origin xyz=0 -0.02 0.074098 rpy=0 0 0, axis -1 0 0, limit lower=0 upper=0.85 effort=50 velocity=2, mimic joint=rightdrive_joint multiplier=1 offset=0
- added joint rightright_outer_knuckle_joint: type revolute, parent rightxarm_gripper_base_link, child rightright_outer_knuckle, origin xyz=0 -0.035 0.059098 rpy=0 0 0, axis -1 0 0, limit lower=0 upper=0.85 effort=50 velocity=2, mimic joint=rightdrive_joint multiplier=1 offset=0
- added joint rightworld_joint: type fixed, parent right_arm_mount, child rightlink_base, origin xyz=0 0 0 rpy=0 0 0
