Commit message: Fixed naming conventions to reflect current setup of arms and fixed chest camera joint

File: dim_cpp/urdf/alfred_base_descr.urdf (robot description, URDF)
Before this commit: robot alfred_base_descr, 63 links, 62 joints
Links:
- removed link leftleft_finger
- removed link leftleft_inner_knuckle
- removed link leftleft_outer_knuckle
- removed link leftlink1
- removed link leftlink2
- removed link leftlink3
- removed link leftlink4
- removed link leftlink5
- removed link leftlink6
- removed link leftlink_base
- removed link leftlink_eef
- removed link leftlink_tcp
- removed link leftright_finger
- removed link leftright_inner_knuckle
- removed link leftright_outer_knuckle
- removed link leftxarm_gripper_base_link
- removed link rightleft_finger
- removed link rightleft_inner_knuckle
- removed link rightleft_outer_knuckle
- removed link rightlink1
- removed link rightlink2
- removed link rightlink3
- removed link rightlink4
- removed link rightlink5
- removed link rightlink6
- removed link rightlink7
- removed link rightlink_base
- removed link rightlink_eef
- removed link rightlink_tcp
- removed link rightright_finger
- removed link rightright_inner_knuckle
- removed link rightright_outer_knuckle
- removed link rightxarm_gripper_base_link
- added link left_left_finger, mass 0.048304; collision mesh filename=package://xarm_description/meshes/gripper/xarm/left_finger.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; visual mesh filename=package://xarm_description/meshes/gripper/xarm/left_finger.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
- added link left_left_inner_knuckle, mass 0.0230125781256706; collision mesh filename=package://xarm_description/meshes/gripper/xarm/left_inner_k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; visual mesh filename=package://xarm_description/meshes/gripper/xarm/left_inner_k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
- added link left_left_outer_knuckle, mass 0.033618; collision mesh filename=package://xarm_description/meshes/gripper/xarm/left_outer_k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; visual mesh filename=package://xarm_description/meshes/gripper/xarm/left_outer_k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
- added link left_link1, mass 2.382; collision mesh filename=package://xarm_description/meshes/xarm7/visual/link1.stl; visual mesh filename=package://xarm_description/meshes/xarm7/visual/link1.stl
- added link left_link2, mass 1.869; collision mesh filename=package://xarm_description/meshes/xarm7/visual/link2.stl; visual mesh filename=package://xarm_description/meshes/xarm7/visual/link2.stl
- added link left_link3, mass 1.6383; collision mesh filename=package://xarm_description/meshes/xarm7/visual/link3.stl; visual mesh filename=package://xarm_description/meshes/xarm7/visual/link3.stl
- added link left_link4, mass 1.7269; collision mesh filename=package://xarm_description/meshes/xarm7/visual/link4.stl; visual mesh filename=package://xarm_description/meshes/xarm7/visual/link4.stl
- added link left_link5, mass 1.3203; collision mesh filename=package://xarm_description/meshes/xarm7/visual/link5.stl; visual mesh filename=package://xarm_description/meshes/xarm7/visual/link5.stl
- added link left_link6, mass 1.325; collision mesh filename=package://xarm_description/meshes/xarm7/visual/link6.stl; visual mesh filename=package://xarm_description/meshes/xarm7/visual/link6.stl
- added link left_link7, mass 0.17; collision mesh filename=package://xarm_description/meshes/end_tool/collision/end_to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; visual mesh filename=package://xarm_description/meshes/xarm7/visual/link7.stl
- added link left_link_base, mass 0.88556; collision mesh filename=package://xarm_description/meshes/xarm7/visual/link_base.stl; visual mesh filename=package://xarm_description/meshes/xarm7/visual/link_base.stl
- added link left_link_eef
- added link left_link_tcp
- added link left_right_finger, mass 0.048304; collision mesh filename=package://xarm_description/meshes/gripper/xarm/right_finger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; visual mesh filename=package://xarm_description/meshes/gripper/xarm/right_finger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
- added link left_right_inner_knuckle, mass 0.023013; collision mesh filename=package://xarm_description/meshes/gripper/xarm/right_inner_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; visual mesh filename=package://xarm_description/meshes/gripper/xarm/right_inner_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
- added link left_right_outer_knuckle, mass 0.033618; collision mesh filename=package://xarm_description/meshes/gripper/xarm/right_outer_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; visual mesh filename=package://xarm_description/meshes/gripper/xarm/right_outer_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
- added link left_xarm_gripper_base_link, mass 0.54156; collision mesh filename=package://xarm_description/meshes/gripper/xarm/base_link.stl; visual mesh filename=package://xarm_description/meshes/gripper/xarm/base_link.stl
- added link right_left_finger, mass 0.048304; collision mesh filename=package://xarm_description/meshes/gripper/xarm/left_finger.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; visual mesh filename=package://xarm_description/meshes/gripper/xarm/left_finger.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
- added link right_left_inner_knuckle, mass 0.0230125781256706; collision mesh filename=package://xarm_description/meshes/gripper/xarm/left_inner_k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; visual mesh filename=package://xarm_description/meshes/gripper/xarm/left_inner_k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
- added link right_left_outer_knuckle, mass 0.033618; collision mesh filename=package://xarm_description/meshes/gripper/xarm/left_outer_k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; visual mesh filename=package://xarm_description/meshes/gripper/xarm/left_outer_k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
- added link right_link1, mass 2.3814; collision mesh filename=package://xarm_description/meshes/xarm6/visual/link1.stl; visual mesh filename=package://xarm_description/meshes/xarm6/visual/link1.stl
- added link right_link2, mass 2.2675; collision mesh filename=package://xarm_description/meshes/xarm6/visual/link2.stl; visual mesh filename=package://xarm_description/meshes/xarm6/visual/link2.stl
- added link right_link3, mass 1.875; collision mesh filename=package://xarm_description/meshes/xarm6/visual/link3.stl; visual mesh filename=package://xarm_description/meshes/xarm6/visual/link3.stl
- added link right_link4, mass 1.3192; collision mesh filename=package://xarm_description/meshes/xarm6/visual/link4.stl; visual mesh filename=package://xarm_description/meshes/xarm6/visual/link4.stl
- added link right_link5, mass 1.33854; collision mesh filename=package://xarm_description/meshes/xarm6/visual/link5.stl; visual mesh filename=package://xarm_description/meshes/xarm6/visual/link5.stl
- added link right_link6, mass 0.17; collision mesh filename=package://xarm_description/meshes/end_tool/collision/end_to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; visual mesh filename=package://xarm_description/meshes/xarm6/visual/link6.stl
- added link right_link_base, mass 2.7; collision mesh filename=package://xarm_description/meshes/xarm6/visual/link_base.stl; visual mesh filename=package://xarm_description/meshes/xarm6/visual/link_base.stl
- added link right_link_eef
- added link right_link_tcp
- added link right_right_finger, mass 0.048304; collision mesh filename=package://xarm_description/meshes/gripper/xarm/right_finger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; visual mesh filename=package://xarm_description/meshes/gripper/xarm/right_finger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
- added link right_right_inner_knuckle, mass 0.023013; collision mesh filename=package://xarm_description/meshes/gripper/xarm/right_inner_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; visual mesh filename=package://xarm_description/meshes/gripper/xarm/right_inner_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
- added link right_right_outer_knuckle, mass 0.033618; collision mesh filename=package://xarm_description/meshes/gripper/xarm/right_outer_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; visual mesh filename=package://xarm_description/meshes/gripper/xarm/right_outer_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
- added link right_xarm_gripper_base_link, mass 0.54156; collision mesh filename=package://xarm_description/meshes/gripper/xarm/base_link.stl; visual mesh filename=package://xarm_description/meshes/gripper/xarm/base_link.stl
Joints:
- removed joint camera_holder_joint
- removed joint leftdrive_joint
- removed joint leftgripper_fix
- removed joint leftjoint1
- removed joint leftjoint2
- removed joint leftjoint3
- removed joint leftjoint4
- removed joint leftjoint5
- removed joint leftjoint6
- removed joint leftjoint_eef
- removed joint leftjoint_tcp
- removed joint leftleft_finger_joint
- removed joint leftleft_inner_knuckle_joint
- removed joint leftright_finger_joint
- removed joint leftright_inner_knuckle_joint
- removed joint leftright_outer_knuckle_joint
- removed joint leftworld_joint
- removed joint rightdrive_joint
- removed joint rightgripper_fix
- removed joint rightjoint1
- removed joint rightjoint2
- removed joint rightjoint3
- removed joint rightjoint4
- removed joint rightjoint5
- removed joint rightjoint6
- removed joint rightjoint7
- removed joint rightjoint_eef
- removed joint rightjoint_tcp
- removed joint rightleft_finger_joint
- removed joint rightleft_inner_knuckle_joint
- removed joint rightright_finger_joint
- removed joint rightright_inner_knuckle_joint
- removed joint rightright_outer_knuckle_joint
- removed joint rightworld_joint
- removed joint tilt_base_joint
- added joint left_drive_joint: type revolute, parent left_xarm_gripper_base_link, child left_left_outer_knuckle, origin xyz=0 0.035 0.059098 rpy=0 0 0, axis 1 0 0, limit lower=0 upper=0.85 effort=50 velocity=2
- added joint left_gripper_fix: type fixed, parent left_link_eef, child left_xarm_gripper_base_link, origin xyz=0 0 0 rpy=0 0 0
- added joint left_joint1: type revolute, parent left_link_base, child left_link1, origin xyz=0 0 0.267 rpy=0 0 0, axis 0 0 1, limit lower=-6.283185307179586 upper=6.283185307179586 effort=50 velocity=3.14
- added joint left_joint2: type revolute, parent left_link1, child left_link2, origin xyz=0 0 0 rpy=-1.5708 0 0, axis 0 0 1, limit lower=-2.059 upper=2.0944 effort=50 velocity=3.14
- added joint left_joint3: type revolute, parent left_link2, child left_link3, origin xyz=0 -0.293 0 rpy=1.5708 0 0, axis 0 0 1, limit lower=-6.283185307179586 upper=6.283185307179586 effort=30 velocity=3.14
- added joint left_joint4: type revolute, parent left_link3, child left_link4, origin xyz=0.0525 0 0 rpy=1.5708 0 0, axis 0 0 1, limit lower=-0.19198 upper=3.927 effort=30 velocity=3.14
- added joint left_joint5: type revolute, parent left_link4, child left_link5, origin xyz=0.0775 -0.3425 0 rpy=1.5708 0 0, axis 0 0 1, limit lower=-6.283185307179586 upper=6.283185307179586 effort=30 velocity=3.14
- added joint left_joint6: type revolute, parent left_link5, child left_link6, origin xyz=0 0 0 rpy=1.5708 0 0, axis 0 0 1, limit lower=-1.69297 upper=3.141592653589793 effort=20 velocity=3.14
- added joint left_joint7: type revolute, parent left_link6, child left_link7, origin xyz=0.076 0.097 0 rpy=-1.5708 0 0, axis 0 0 1, limit lower=-6.283185307179586 upper=6.283185307179586 effort=20 velocity=3.14
- added joint left_joint_eef: type fixed, parent left_link7, child left_link_eef, origin xyz=0 0 0 rpy=0 0 0
- added joint left_joint_tcp: type fixed, parent left_xarm_gripper_base_link, child left_link_tcp, origin xyz=0 0 0.172 rpy=0 0 0
- added joint left_left_finger_joint: type revolute, parent left_left_outer_knuckle, child left_left_finger, origin xyz=0 0.035465 0.042039 rpy=0 0 0, axis -1 0 0, limit lower=0 upper=0.85 effort=50 velocity=2, mimic joint=left_drive_joint multiplier=1 offset=0
- added joint left_left_inner_knuckle_joint: type revolute, parent left_xarm_gripper_base_link, child left_left_inner_knuckle, origin xyz=0 0.02 0.074098 rpy=0 0 0, axis 1 0 0, limit lower=0 upper=0.85 effort=50 velocity=2, mimic joint=left_drive_joint multiplier=1 offset=0
- added joint left_right_finger_joint: type revolute, parent left_right_outer_knuckle, child left_right_finger, origin xyz=0 -0.035465 0.042039 rpy=0 0 0, axis 1 0 0, limit lower=0 upper=0.85 effort=50 velocity=2, mimic joint=left_drive_joint multiplier=1 offset=0
- added joint left_right_inner_knuckle_joint: type revolute, parent left_xarm_gripper_base_link, child left_right_inner_knuckle, origin xyz=0 -0.02 0.074098 rpy=0 0 0, axis -1 0 0, limit lower=0 upper=0.85 effort=50 velocity=2, mimic joint=left_drive_joint multiplier=1 offset=0
- added joint left_right_outer_knuckle_joint: type revolute, parent left_xarm_gripper_base_link, child left_right_outer_knuckle, origin xyz=0 -0.035 0.059098 rpy=0 0 0, axis -1 0 0, limit lower=0 upper=0.85 effort=50 velocity=2, mimic joint=left_drive_joint multiplier=1 offset=0
- added joint left_world_joint: type fixed, parent left_arm_mount, child left_link_base, origin xyz=0 0 0 rpy=0 0 0
- added joint pan_joint: type revolute, parent alfred_base_link, child tilt_base, origin xyz=.225 -.365 1.645 rpy=0 0 0, axis 0 0 1, limit lower=-1.57 upper=1.57 effort=100 velocity=0.1
- added joint right_drive_joint: type revolute, parent right_xarm_gripper_base_link, child right_left_outer_knuckle, origin xyz=0 0.035 0.059098 rpy=0 0 0, axis 1 0 0, limit lower=0 upper=0.85 effort=50 velocity=2
- added joint right_gripper_fix: type fixed, parent right_link_eef, child right_xarm_gripper_base_link, origin xyz=0 0 0 rpy=0 0 0
- added joint right_joint1: type revolute, parent right_link_base, child right_link1, origin xyz=0 0 0.267 rpy=0 0 0, axis 0 0 1, limit lower=-6.283185307179586 upper=6.283185307179586 effort=50.0 velocity=3.14
- added joint right_joint2: type revolute, parent right_link1, child right_link2, origin xyz=0 0 0 rpy=-1.5708 0 0, axis 0 0 1, limit lower=-2.059 upper=2.0944 effort=50.0 velocity=3.14
- added joint right_joint3: type revolute, parent right_link2, child right_link3, origin xyz=0.0535 -0.2845 0 rpy=0 0 0, axis 0 0 1, limit lower=-3.927 upper=0.19198 effort=32.0 velocity=3.14
- added joint right_joint4: type revolute, parent right_link3, child right_link4, origin xyz=0.0775 0.3425 0 rpy=-1.5708 0 0, axis 0 0 1, limit lower=-6.283185307179586 upper=6.283185307179586 effort=32.0 velocity=3.14
- added joint right_joint5: type revolute, parent right_link4, child right_link5, origin xyz=0 0 0 rpy=1.5708 0 0, axis 0 0 1, limit lower=-1.69297 upper=3.141592653589793 effort=32.0 velocity=3.14
- added joint right_joint6: type revolute, parent right_link5, child right_link6, origin xyz=0.076 0.097 0 rpy=-1.5708 0 0, axis 0 0 1, limit lower=-6.283185307179586 upper=6.283185307179586 effort=20.0 velocity=3.14
- added joint right_joint_eef: type fixed, parent right_link6, child right_link_eef, origin xyz=0 0 0 rpy=0 0 0
- added joint right_joint_tcp: type fixed, parent right_xarm_gripper_base_link, child right_link_tcp, origin xyz=0 0 0.172 rpy=0 0 0
- added joint right_left_finger_joint: type revolute, parent right_left_outer_knuckle, child right_left_finger, origin xyz=0 0.035465 0.042039 rpy=0 0 0, axis -1 0 0, limit lower=0 upper=0.85 effort=50 velocity=2, mimic joint=right_drive_joint multiplier=1 offset=0
- added joint right_left_inner_knuckle_joint: type revolute, parent right_xarm_gripper_base_link, child right_left_inner_knuckle, origin xyz=0 0.02 0.074098 rpy=0 0 0, axis 1 0 0, limit lower=0 upper=0.85 effort=50 velocity=2, mimic joint=right_drive_joint multiplier=1 offset=0
- added joint right_right_finger_joint: type revolute, parent right_right_outer_knuckle, child right_right_finger, origin xyz=0 -0.035465 0.042039 rpy=0 0 0, axis 1 0 0, limit lower=0 upper=0.85 effort=50 velocity=2, mimic joint=right_drive_joint multiplier=1 offset=0
- added joint right_right_inner_knuckle_joint: type revolute, parent right_xarm_gripper_base_link, child right_right_inner_knuckle, origin xyz=0 -0.02 0.074098 rpy=0 0 0, axis -1 0 0, limit lower=0 upper=0.85 effort=50 velocity=2, mimic joint=right_drive_joint multiplier=1 offset=0
- added joint right_right_outer_knuckle_joint: type revolute, parent right_xarm_gripper_base_link, child right_right_outer_knuckle, origin xyz=0 -0.035 0.059098 rpy=0 0 0, axis -1 0 0, limit lower=0 upper=0.85 effort=50 velocity=2, mimic joint=right_drive_joint multiplier=1 offset=0
- added joint right_world_joint: type fixed, parent right_arm_mount, child right_link_base, origin xyz=0 0 0 rpy=0 0 0
- added joint tilt_joint: type revolute, parent tilt_base, child camera_holder, origin xyz=0 0 0.014 rpy=0 0 0, axis 1 0 0, limit lower=-1.57 upper=1.57 effort=100 velocity=0.1
- joint chest_cam_joint: parent alfred_base_link -> pillar_platform
- joint left_arm_mount_joint: origin xyz=.12325 -.319646 1.4125 rpy=1.57079633 0 -1.57079633 -> xyz=.32675 -.319646 1.4125 rpy=1.57079633 3.14159265 1.57079633
- joint left_wheel_joint: origin xyz=-0.0561 -0.395 -0.0375 rpy=0 0 -1.5707 -> xyz=0.5061 -0.395 -0.0375 rpy=0 0 1.5707
- joint right_arm_mount_joint: origin xyz=.32675 -.319646 1.4125 rpy=1.57079633 3.14159265 1.57079633 -> xyz=.12325 -.319646 1.4125 rpy=1.57079633 0 -1.57079633
- joint right_wheel_joint: origin xyz=0.5061 -0.395 -0.0375 rpy=0 0 1.5707 -> xyz=-0.0561 -0.395 -0.0375 rpy=0 0 -1.5707

File: dim_cpp/urdf/alfred_base_descr.urdf.xacro (robot description, xacro)
@@ -15,5 +15,5 @@
 	<!-- load xarm6 device -->
 	<xacro:include filename="$(find xarm_description)/urdf/xarm_device_macro.xacro" />
-	<xacro:xarm_device prefix="left" hw_ns="xarm" limited="false"
+	<xacro:xarm_device prefix="right_" hw_ns="xarm" limited="false"
 		effort_control="false" velocity_control="false"
 		add_gripper="true" add_vacuum_gripper="false"
@@ -32,7 +32,7 @@
 		robot_ip="192.168.1.210" report_type="dev"
 		baud_checkset="true" default_gripper_baud="2000000"
-		model1300="false" attach_to="left_arm_mount" attach_xyz="0 0 0" attach_rpy="0 0 0"
+		model1300="false" attach_to="right_arm_mount" attach_xyz="0 0 0" attach_rpy="0 0 0"
 		robot_sn="" use_gazebo_camera="false" mesh_suffix="stl" kinematics_suffix="" />
-	<xacro:xarm_device prefix="right" hw_ns="xarm" limited="false"
+	<xacro:xarm_device prefix="left_" hw_ns="xarm" limited="false"
 		effort_control="false" velocity_control="false"
 		add_gripper="true" add_vacuum_gripper="false"
@@ -51,5 +51,5 @@
 		robot_ip="192.168.1.211" report_type="dev"
 		baud_checkset="true" default_gripper_baud="2000000"
-		model1300="false" attach_to="right_arm_mount" attach_xyz="0 0 0" attach_rpy="0 0 0"
+		model1300="false" attach_to="left_arm_mount" attach_xyz="0 0 0" attach_rpy="0 0 0"
 		robot_sn="" use_gazebo_camera="false" mesh_suffix="stl" kinematics_suffix="" />
 </robot>

File: dim_cpp/urdf/include/alfred_base.urdf.xacro (robot description, xacro)
@@ -43,5 +43,5 @@
             <origin xyz="-.225 .2125 .1232" rpy="0 0 0" />
         </joint>
-        <link name="botwheel_left">
+        <link name="botwheel_right">
             <visual>
                 <origin xyz="0 0 0" rpy="0 0 0" />
@@ -67,11 +67,11 @@
             </inertial>
         </link>
-        <joint name="left_wheel_joint" type="continuous">
-            <parent link="alfred_base_link" />
-            <child link="botwheel_left" />
+        <joint name="right_wheel_joint" type="continuous">
+            <parent link="alfred_base_link" />
+            <child link="botwheel_right" />
             <origin xyz="-0.0561 -0.395 -0.0375" rpy="0 0 -1.5707" />
             <axis xyz="0 1 0" />
         </joint>
-        <link name="botwheel_right">
+        <link name="botwheel_left">
             <visual>
                 <origin xyz="0 0 0" rpy="0 0 0" />
@@ -97,7 +97,7 @@
             </inertial>
         </link>
-        <joint name="right_wheel_joint" type="continuous">
-            <parent link="alfred_base_link" />
-            <child link="botwheel_right" />
+        <joint name="left_wheel_joint" type="continuous">
+            <parent link="alfred_base_link" />
+            <child link="botwheel_left" />
             <origin xyz="0.5061 -0.395 -0.0375" rpy="0 0 1.5707" />
             <axis xyz="0 1 0" />
@@ -159,5 +159,5 @@
             </inertial>
         </link>
-        <joint name="tilt_base_joint" type="revolute">
+        <joint name="pan_joint" type="revolute">
             <parent link="alfred_base_link" />
             <child link="tilt_base" />
@@ -191,5 +191,5 @@
             </inertial>
         </link>
-        <joint name="camera_holder_joint" type="revolute">
+        <joint name="tilt_joint" type="revolute">
             <parent link="tilt_base" />
             <child link="camera_holder" />
@@ -206,7 +206,13 @@
         <link name="chest_cam_link" />
         <joint name="chest_cam_joint" type="fixed">
-            <parent link="alfred_base_link" />
+            <parent link="pillar_platform" />
             <child link="chest_cam_link" />
             <origin xyz=".225 -.455681 1.441731" rpy="0.78539816 0 0" />
+        </joint>
+        <link name="right_arm_mount" />
+        <joint name="right_arm_mount_joint" type="fixed">
+            <parent link="pillar_platform" />
+            <child link="right_arm_mount" />
+            <origin xyz=".12325 -.319646 1.4125" rpy="1.57079633 0 -1.57079633" />
         </joint>
         <link name="left_arm_mount" />
@@ -214,10 +220,4 @@
             <parent link="pillar_platform" />
             <child link="left_arm_mount" />
-            <origin xyz=".12325 -.319646 1.4125" rpy="1.57079633 0 -1.57079633" />
-        </joint>
-        <link name="right_arm_mount" />
-        <joint name="right_arm_mount_joint" type="fixed">
-            <parent link="pillar_platform" />
-            <child link="right_arm_mount" />
             <origin xyz=".32675 -.319646 1.4125" rpy="1.57079633 3.14159265 1.57079633" />
         </joint>

Commit message: Changed world to local_world

File: dim_cpp/urdf/alfred_base_descr.urdf (robot description, URDF)
Before this commit: robot alfred_base_descr, 63 links, 62 joints
Links:
- removed link world
- added link local_world
Joints:
- joint base_parent_joint: parent world -> local_world
- joint right_drive_joint: limit lower=0 upper=0.85 effort=50 velocity=2 -> lower=0.0 upper=0.85 effort=50 velocity=2.0
- joint right_left_finger_joint: limit lower=0 upper=0.85 effort=50 velocity=2 -> lower=0.0 upper=0.85 effort=50 velocity=2.0

File: dim_cpp/urdf/alfred_base_descr.urdf.xacro (robot description, xacro)
@@ -2,6 +2,6 @@
 <robot name="alfred_base_descr" xmlns:xacro="http://ros.org/wiki/xacro">
 	<xacro:include filename="$(find dim_cpp)/urdf/include/alfred_base.urdf.xacro" />
-	<link name="world" />
-	<xacro:alfred_base base_frame="world" base_pos_x="0.0" base_pos_y="0.0" base_pos_z="0.0" base_roll="0.0" base_pitch="0.0" base_yaw="0.0" r="0.8" g="0.8" b="0.8" a="1.0" />
+	<link name="local_world" />
+	<xacro:alfred_base base_frame="local_world" base_pos_x="0.0" base_pos_y="0.0" base_pos_z="0.0" base_roll="0.0" base_pitch="0.0" base_yaw="0.0" r="0.8" g="0.8" b="0.8" a="1.0" />
 	<xacro:include filename="$(find depthai_descriptions)/urdf/include/depthai_macro.urdf.xacro" />
 	<xacro:depthai_camera camera_name="head_cam" parent="head_cam_link"
@@ -19,6 +19,6 @@
 		add_gripper="true" add_vacuum_gripper="false"
 		add_bio_gripper="false" dof="6"
-		ros2_control_plugin="uf_robot_hardware/UFRobotSystemHardware" robot_type="xarm"
-		load_gazebo_plugin="false" ros2_control_params=""
+		ros2_control_plugin="uf_robot_hardware/UFRobotFakeSystemHardware" robot_type="xarm"
+		load_gazebo_plugin="true" ros2_control_params=""
 		add_realsense_d435i="false"
 		add_d435i_links="true"
@@ -38,5 +38,5 @@
 		add_gripper="true" add_vacuum_gripper="false"
 		add_bio_gripper="false" dof="7"
-		ros2_control_plugin="uf_robot_hardware/UFRobotSystemHardware" robot_type="xarm"
+		ros2_control_plugin="uf_robot_hardware/UFRobotFakeSystemHardware" robot_type="xarm"
 		load_gazebo_plugin="false" ros2_control_params=""
 		add_realsense_d435i="false"
