Commit message: Reversed direction of arms on alfred

File: dim_cpp/urdf/alfred_base_descr.urdf (robot description, URDF)
Before this commit: robot alfred_base_descr, 63 links, 62 joints
Links:
- removed link left_link7
- added link right_link7, mass 0.17; collision mesh filename=package://xarm_description/meshes/end_tool/collision/end_to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; visual mesh filename=package://xarm_description/meshes/xarm7/visual/link7.stl
- link left_link1: mass 2.382 -> 2.3814; geometry collision mesh filename=package://xarm_description/meshes/xarm6/visual/link1.stl; visual mesh filename=package://xarm_description/meshes/xarm6/visual/link1.stl
- link left_link2: mass 1.869 -> 2.2675; geometry collision mesh filename=package://xarm_description/meshes/xarm6/visual/link2.stl; visual mesh filename=package://xarm_description/meshes/xarm6/visual/link2.stl
- link left_link3: mass 1.6383 -> 1.875; geometry collision mesh filename=package://xarm_description/meshes/xarm6/visual/link3.stl; visual mesh filename=package://xarm_description/meshes/xarm6/visual/link3.stl
- link left_link4: mass 1.7269 -> 1.3192; geometry collision mesh filename=package://xarm_description/meshes/xarm6/visual/link4.stl; visual mesh filename=package://xarm_description/meshes/xarm6/visual/link4.stl
- link left_link5: mass 1.3203 -> 1.33854; geometry collision mesh filename=package://xarm_description/meshes/xarm6/visual/link5.stl; visual mesh filename=package://xarm_description/meshes/xarm6/visual/link5.stl
- link left_link6: mass 1.325 -> 0.17; geometry collision mesh filename=package://xarm_description/meshes/end_tool/collision/end_to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; visual mesh filename=package://xarm_description/meshes/xarm6/visual/link6.stl
- link left_link_base: mass 0.88556 -> 2.7; geometry collision mesh filename=package://xarm_description/meshes/xarm6/visual/link_base.stl; visual mesh filename=package://xarm_description/meshes/xarm6/visual/link_base.stl
- link right_link1: mass 2.3814 -> 2.382; geometry collision mesh filename=package://xarm_description/meshes/xarm7/visual/link1.stl; visual mesh filename=package://xarm_description/meshes/xarm7/visual/link1.stl
- link right_link2: mass 2.2675 -> 1.869; geometry collision mesh filename=package://xarm_description/meshes/xarm7/visual/link2.stl; visual mesh filename=package://xarm_description/meshes/xarm7/visual/link2.stl
- link right_link3: mass 1.875 -> 1.6383; geometry collision mesh filename=package://xarm_description/meshes/xarm7/visual/link3.stl; visual mesh filename=package://xarm_description/meshes/xarm7/visual/link3.stl
- link right_link4: mass 1.3192 -> 1.7269; geometry collision mesh filename=package://xarm_description/meshes/xarm7/visual/link4.stl; visual mesh filename=package://xarm_description/meshes/xarm7/visual/link4.stl
- link right_link5: mass 1.33854 -> 1.3203; geometry collision mesh filename=package://xarm_description/meshes/xarm7/visual/link5.stl; visual mesh filename=package://xarm_description/meshes/xarm7/visual/link5.stl
- link right_link6: mass 0.17 -> 1.325; geometry collision mesh filename=package://xarm_description/meshes/xarm7/visual/link6.stl; visual mesh filename=package://xarm_description/meshes/xarm7/visual/link6.stl
- link right_link_base: mass 2.7 -> 0.88556; geometry collision mesh filename=package://xarm_description/meshes/xarm7/visual/link_base.stl; visual mesh filename=package://xarm_description/meshes/xarm7/visual/link_base.stl
Joints:
- removed joint left_joint7
- added joint right_joint7: type revolute, parent right_link6, child right_link7, origin xyz=0.076 0.097 0 rpy=-1.5708 0 0, axis 0 0 1, limit lower=-6.283185307179586 upper=6.283185307179586 effort=20 velocity=3.14
- joint left_joint1: limit lower=-6.283185307179586 upper=6.283185307179586 effort=50 velocity=3.14 -> lower=-6.283185307179586 upper=6.283185307179586 effort=50.0 velocity=3.14
- joint left_joint2: limit lower=-2.059 upper=2.0944 effort=50 velocity=3.14 -> lower=-2.059 upper=2.0944 effort=50.0 velocity=3.14
- joint left_joint3: limit lower=-6.283185307179586 upper=6.283185307179586 effort=30 velocity=3.14 -> lower=-3.927 upper=0.19198 effort=32.0 velocity=3.14; origin xyz=0 -0.293 0 rpy=1.5708 0 0 -> xyz=0.0535 -0.2845 0 rpy=0 0 0
- joint left_joint4: limit lower=-0.19198 upper=3.927 effort=30 velocity=3.14 -> lower=-6.283185307179586 upper=6.283185307179586 effort=32.0 velocity=3.14; origin xyz=0.0525 0 0 rpy=1.5708 0 0 -> xyz=0.0775 0.3425 0 rpy=-1.5708 0 0
- joint left_joint5: limit lower=-6.283185307179586 upper=6.283185307179586 effort=30 velocity=3.14 -> lower=-1.69297 upper=3.141592653589793 effort=32.0 velocity=3.14; origin xyz=0.0775 -0.3425 0 rpy=1.5708 0 0 -> xyz=0 0 0 rpy=1.5708 0 0
- joint left_joint6: limit lower=-1.69297 upper=3.141592653589793 effort=20 velocity=3.14 -> lower=-6.283185307179586 upper=6.283185307179586 effort=20.0 velocity=3.14; origin xyz=0 0 0 rpy=1.5708 0 0 -> xyz=0.076 0.097 0 rpy=-1.5708 0 0
- joint left_joint_eef: parent left_link7 -> left_link6
- joint right_drive_joint: limit lower=0.0 upper=0.85 effort=50 velocity=2.0 -> lower=0 upper=0.85 effort=50 velocity=2
- joint right_joint1: limit lower=-6.283185307179586 upper=6.283185307179586 effort=50.0 velocity=3.14 -> lower=-6.283185307179586 upper=6.283185307179586 effort=50 velocity=3.14
- joint right_joint2: limit lower=-2.059 upper=2.0944 effort=50.0 velocity=3.14 -> lower=-2.059 upper=2.0944 effort=50 velocity=3.14
- joint right_joint3: limit lower=-3.927 upper=0.19198 effort=32.0 velocity=3.14 -> lower=-6.283185307179586 upper=6.283185307179586 effort=30 velocity=3.14; origin xyz=0.0535 -0.2845 0 rpy=0 0 0 -> xyz=0 -0.293 0 rpy=1.5708 0 0
- joint right_joint4: limit lower=-6.283185307179586 upper=6.283185307179586 effort=32.0 velocity=3.14 -> lower=-0.19198 upper=3.927 effort=30 velocity=3.14; origin xyz=0.0775 0.3425 0 rpy=-1.5708 0 0 -> xyz=0.0525 0 0 rpy=1.5708 0 0
- joint right_joint5: limit lower=-1.69297 upper=3.141592653589793 effort=32.0 velocity=3.14 -> lower=-6.283185307179586 upper=6.283185307179586 effort=30 velocity=3.14; origin xyz=0 0 0 rpy=1.5708 0 0 -> xyz=0.0775 -0.3425 0 rpy=1.5708 0 0
- joint right_joint6: limit lower=-6.283185307179586 upper=6.283185307179586 effort=20.0 velocity=3.14 -> lower=-1.69297 upper=3.141592653589793 effort=20 velocity=3.14; origin xyz=0.076 0.097 0 rpy=-1.5708 0 0 -> xyz=0 0 0 rpy=1.5708 0 0
- joint right_joint_eef: parent right_link6 -> right_link7
- joint right_left_finger_joint: limit lower=0.0 upper=0.85 effort=50 velocity=2.0 -> lower=0 upper=0.85 effort=50 velocity=2

File: dim_cpp/urdf/alfred_base_descr.urdf.xacro (robot description, xacro)
@@ -18,5 +18,5 @@
 		effort_control="false" velocity_control="false"
 		add_gripper="true" add_vacuum_gripper="false"
-		add_bio_gripper="false" dof="6"
+		add_bio_gripper="false" dof="7"
 		ros2_control_plugin="uf_robot_hardware/UFRobotFakeSystemHardware" robot_type="xarm"
 		load_gazebo_plugin="true" ros2_control_params=""
@@ -30,5 +30,5 @@
 		geometry_mesh_origin_xyz="0 0 0" geometry_mesh_origin_rpy="0 0 0"
 		geometry_mesh_tcp_xyz="0 0 0" geometry_mesh_tcp_rpy="0 0 0"
-		robot_ip="192.168.1.210" report_type="dev"
+		robot_ip="192.168.1.197" report_type="dev"
 		baud_checkset="true" default_gripper_baud="2000000"
 		model1300="false" attach_to="right_arm_mount" attach_xyz="0 0 0" attach_rpy="0 0 0"
@@ -37,5 +37,5 @@
 		effort_control="false" velocity_control="false"
 		add_gripper="true" add_vacuum_gripper="false"
-		add_bio_gripper="false" dof="7"
+		add_bio_gripper="false" dof="6"
 		ros2_control_plugin="uf_robot_hardware/UFRobotFakeSystemHardware" robot_type="xarm"
 		load_gazebo_plugin="false" ros2_control_params=""
@@ -49,5 +49,5 @@
 		geometry_mesh_origin_xyz="0 0 0" geometry_mesh_origin_rpy="0 0 0"
 		geometry_mesh_tcp_xyz="0 0 0" geometry_mesh_tcp_rpy="0 0 0"
-		robot_ip="192.168.1.211" report_type="dev"
+		robot_ip="192.168.1.210" report_type="dev"
 		baud_checkset="true" default_gripper_baud="2000000"
 		model1300="false" attach_to="left_arm_mount" attach_xyz="0 0 0" attach_rpy="0 0 0"
