Commit message: URDF with both cameras and xarm6 done- not tested with runner code

File: dim_cpp/urdf/alfred_base_descr.urdf.xacro (robot description, xacro)
@@ -4,3 +4,71 @@
 	<link name="world" />
 	<xacro:alfred_base base_frame="world" base_pos_x="0.0" base_pos_y="0.0" base_pos_z="0.0" base_roll="0.0" base_pitch="0.0" base_yaw="0.0" r="0.8" g="0.8" b="0.8" a="1.0" />
+	<xacro:include filename="$(find depthai_descriptions)/urdf/include/depthai_macro.urdf.xacro" />
+	<xacro:depthai_camera camera_name="head_cam" parent="head_cam_link"
+		camera_model="OAK-D-PRO" base_frame="head_cam_frame"
+		cam_pos_x="0" cam_pos_y="-0.022921" cam_pos_z="0.004764"
+		cam_roll="0" cam_pitch="0" cam_yaw="-1.5707963267948966" />
+	<xacro:depthai_camera camera_name="chest_cam" parent="chest_cam_link"
+		camera_model="OAK-D-PRO" base_frame="chest_cam_frame"
+		cam_pos_x="0" cam_pos_y="-0.022921" cam_pos_z="-0.004764"
+		cam_roll="3.14159265" cam_pitch="0" cam_yaw="-1.5707963267948966" />
+	<xacro:arg name="prefix" default=""/>
+	<xacro:arg name="hw_ns" default="xarm"/>
+	<xacro:arg name="limited" default="false"/>
+	<xacro:arg name="effort_control" default="false"/>
+	<xacro:arg name="velocity_control" default="false"/>
+	<xacro:arg name="add_gripper" default="true"/>
+	<xacro:arg name="add_vacuum_gripper" default="false"/>
+	<xacro:arg name="add_bio_gripper" default="false"/>
+	<xacro:arg name="model1300" default="false"/>
+	<xacro:arg name="dof" default="6"/>
+	<xacro:arg name="robot_ip" default=""/>
+	<xacro:arg name="robot_type" default="xarm"/>
+	<xacro:arg name="robot_sn" default=""/>
+	<xacro:arg name="report_type" default="normal"/>
+	<xacro:arg name="ros2_control_plugin" default="uf_robot_hardware/UFRobotSystemHardware"/>
+	<xacro:arg name="ros2_control_params" default=""/>
+	<xacro:arg name="add_realsense_d435i" default="false"/>
+	<xacro:arg name="add_d435i_links" default="true"/>
+	<xacro:arg name="use_gazebo_camera" default="false"/>
+	<xacro:arg name="add_other_geometry" default="false"/>
+	<xacro:arg name="geometry_type" default="box"/>
+	<xacro:arg name="geometry_mass" default="0.1"/>
+	<xacro:arg name="geometry_height" default="0.1"/>
+	<xacro:arg name="geometry_radius" default="0.1"/>
+	<xacro:arg name="geometry_length" default="0.1"/>
+	<xacro:arg name="geometry_width" default="0.1"/>
+	<xacro:arg name="geometry_mesh_filename" default=""/>
+	<xacro:arg name="geometry_mesh_origin_xyz" default="0 0 0"/>
+	<xacro:arg name="geometry_mesh_origin_rpy" default="0 0 0"/>
+	<xacro:arg name="geometry_mesh_tcp_xyz" default="0 0 0"/>
+	<xacro:arg name="geometry_mesh_tcp_rpy" default="0 0 0"/>
+	<xacro:arg name="baud_checkset" default="true"/>
+	<xacro:arg name="default_gripper_baud" default="2000000"/>
+	<xacro:arg name="attach_to" default="left_arm_mount"/>
+	<xacro:arg name="attach_xyz" default="0 0 0"/>
+	<xacro:arg name="attach_rpy" default="0 0 0"/>
+	<xacro:arg name="mesh_suffix" default="stl"/>
+	<xacro:arg name="kinematics_suffix" default=""/>
+	<!-- load xarm device -->
+	<xacro:include filename="$(find xarm_description)/urdf/xarm_device_macro.xacro" />
+	<xacro:xarm_device prefix="$(arg prefix)" hw_ns="$(arg hw_ns)" limited="$(arg limited)"
+		effort_control="$(arg effort_control)" velocity_control="$(arg velocity_control)"
+		add_gripper="$(arg add_gripper)" add_vacuum_gripper="$(arg add_vacuum_gripper)"
+		add_bio_gripper="$(arg add_bio_gripper)" dof="$(arg dof)"
+		ros2_control_plugin="$(arg ros2_control_plugin)" robot_type="$(arg robot_type)"
+		load_gazebo_plugin="true" ros2_control_params="$(arg ros2_control_params)"
+		add_realsense_d435i="$(arg add_realsense_d435i)"
+		add_d435i_links="$(arg add_d435i_links)"
+		add_other_geometry="$(arg add_other_geometry)"
+		geometry_type="$(arg geometry_type)" geometry_mass="$(arg geometry_mass)"
+		geometry_height="$(arg geometry_height)" geometry_radius="$(arg geometry_radius)"
+		geometry_length="$(arg geometry_length)" geometry_width="$(arg geometry_width)"
+		geometry_mesh_filename="$(arg geometry_mesh_filename)"
+		geometry_mesh_origin_xyz="$(arg geometry_mesh_origin_xyz)" geometry_mesh_origin_rpy="$(arg geometry_mesh_origin_rpy)"
+		geometry_mesh_tcp_xyz="$(arg geometry_mesh_tcp_xyz)" geometry_mesh_tcp_rpy="$(arg geometry_mesh_tcp_rpy)"
+		robot_ip="$(arg robot_ip)" report_type="$(arg report_type)"
+		baud_checkset="$(arg baud_checkset)" default_gripper_baud="$(arg default_gripper_baud)"
+		model1300="$(arg model1300)" attach_to="$(arg attach_to)" attach_xyz="$(arg attach_xyz)" attach_rpy="$(arg attach_rpy)"
+		robot_sn="$(arg robot_sn)" use_gazebo_camera="$(arg use_gazebo_camera)" mesh_suffix="$(arg mesh_suffix)" kinematics_suffix="$(arg kinematics_suffix)" />
 </robot>

File: dim_cpp/urdf/include/alfred_base.urdf.xacro (robot description, xacro)
@@ -198,4 +198,28 @@
             <limit lower="-1.57" upper="1.57" effort="100" velocity="0.1"/>
         </joint>
+        <link name="head_cam_link" />
+        <joint name="head_cam_joint" type="fixed">
+            <parent link="camera_holder" />
+            <child link="head_cam_link" />
+            <origin xyz="0 -0.0025 0.057" rpy="0 0 0" />
+        </joint>
+        <link name="chest_cam_link" />
+        <joint name="chest_cam_joint" type="fixed">
+            <parent link="alfred_base_link" />
+            <child link="chest_cam_link" />
+            <origin xyz=".225 -.455681 1.441731" rpy="0.78539816 0 0" />
+        </joint>
+        <link name="left_arm_mount" />
+        <joint name="left_arm_mount_joint" type="fixed">
+            <parent link="pillar_platform" />
+            <child link="left_arm_mount" />
+            <origin xyz=".12325 -.319646 1.4125" rpy="1.57079633 0 -1.57079633" />
+        </joint>
+        <link name="right_arm_mount" />
+        <joint name="right_arm_mount_joint" type="fixed">
+            <parent link="pillar_platform" />
+            <child link="right_arm_mount" />
+            <origin xyz=".32675 -.319646 1.4125" rpy="-1.57079633 0 1.57079633" />
+        </joint>
     </xacro:macro>
     <!-- <xacro:alfred_base base_frame="world" base_pos_x="0.0" base_pos_y="0.0" base_pos_z="0.0" base_roll="0.0" base_pitch="0.0" base_yaw="0.0" r="0.8" g="0.8" b="0.8" a="1.0" /> -->

File: xarm_ros2/xarm_description/urdf/xarm_device.urdf.xacro (robot description, xacro)
@@ -10,5 +10,5 @@
   <xacro:arg name="add_bio_gripper" default="false"/>
   <xacro:arg name="model1300" default="false"/>
-  <xacro:arg name="dof" default="7"/>
+  <xacro:arg name="dof" default="6"/>
   <xacro:arg name="robot_ip" default=""/>
   <xacro:arg name="robot_type" default="xarm"/>
@@ -60,19 +60,3 @@
     model1300="$(arg model1300)" attach_to="$(arg attach_to)" attach_xyz="$(arg attach_xyz)" attach_rpy="$(arg attach_rpy)"
     robot_sn="$(arg robot_sn)" use_gazebo_camera="$(arg use_gazebo_camera)" mesh_suffix="$(arg mesh_suffix)" kinematics_suffix="$(arg kinematics_suffix)" />
-	<xacro:arg name="camera_name" default="oak" />
-	<xacro:arg name="camera_model" default="OAK-D-PRO" />
-	<xacro:arg name="base_frame" default="oak-d_frame" />
-	<xacro:arg name="parent_frame" default="link6" />
-	<xacro:arg name="cam_pos_x" default="0.0875" />
-	<xacro:arg name="cam_pos_y" default="0.0" />
-	<xacro:arg name="cam_pos_z" default="0.02792" />
-	<xacro:arg name="cam_roll" default="3.141592653589793" />
-	<xacro:arg name="cam_pitch" default="-1.5707963267948966" />
-	<xacro:arg name="cam_yaw" default="0.0" />
-	<xacro:arg name="rs_compat" default="false" />
-	<xacro:include filename="$(find depthai_descriptions)/urdf/include/depthai_macro.urdf.xacro" />
-	<xacro:depthai_camera camera_name="$(arg camera_name)" parent="$(arg parent_frame)"
-		camera_model="$(arg camera_model)" base_frame="$(arg base_frame)"
-		cam_pos_x="$(arg cam_pos_x)" cam_pos_y="$(arg cam_pos_y)" cam_pos_z="$(arg cam_pos_z)"
-		cam_roll="$(arg cam_roll)" cam_pitch="$(arg cam_pitch)" cam_yaw="$(arg cam_yaw)" />
 </robot>

Commit message: Added second arm

File: dim_cpp/urdf/alfred_base_descr.urdf.xacro (robot description, xacro)
@@ -13,62 +13,43 @@
 		cam_pos_x="0" cam_pos_y="-0.022921" cam_pos_z="-0.004764"
 		cam_roll="3.14159265" cam_pitch="0" cam_yaw="-1.5707963267948966" />
-	<xacro:arg name="prefix" default=""/>
-	<xacro:arg name="hw_ns" default="xarm"/>
-	<xacro:arg name="limited" default="false"/>
-	<xacro:arg name="effort_control" default="false"/>
-	<xacro:arg name="velocity_control" default="false"/>
-	<xacro:arg name="add_gripper" default="true"/>
-	<xacro:arg name="add_vacuum_gripper" default="false"/>
-	<xacro:arg name="add_bio_gripper" default="false"/>
-	<xacro:arg name="model1300" default="false"/>
-	<xacro:arg name="dof" default="6"/>
-	<xacro:arg name="robot_ip" default=""/>
-	<xacro:arg name="robot_type" default="xarm"/>
-	<xacro:arg name="robot_sn" default=""/>
-	<xacro:arg name="report_type" default="normal"/>
-	<xacro:arg name="ros2_control_plugin" default="uf_robot_hardware/UFRobotSystemHardware"/>
-	<xacro:arg name="ros2_control_params" default=""/>
-	<xacro:arg name="add_realsense_d435i" default="false"/>
-	<xacro:arg name="add_d435i_links" default="true"/>
-	<xacro:arg name="use_gazebo_camera" default="false"/>
-	<xacro:arg name="add_other_geometry" default="false"/>
-	<xacro:arg name="geometry_type" default="box"/>
-	<xacro:arg name="geometry_mass" default="0.1"/>
-	<xacro:arg name="geometry_height" default="0.1"/>
-	<xacro:arg name="geometry_radius" default="0.1"/>
-	<xacro:arg name="geometry_length" default="0.1"/>
-	<xacro:arg name="geometry_width" default="0.1"/>
-	<xacro:arg name="geometry_mesh_filename" default=""/>
-	<xacro:arg name="geometry_mesh_origin_xyz" default="0 0 0"/>
-	<xacro:arg name="geometry_mesh_origin_rpy" default="0 0 0"/>
-	<xacro:arg name="geometry_mesh_tcp_xyz" default="0 0 0"/>
-	<xacro:arg name="geometry_mesh_tcp_rpy" default="0 0 0"/>
-	<xacro:arg name="baud_checkset" default="true"/>
-	<xacro:arg name="default_gripper_baud" default="2000000"/>
-	<xacro:arg name="attach_to" default="left_arm_mount"/>
-	<xacro:arg name="attach_xyz" default="0 0 0"/>
-	<xacro:arg name="attach_rpy" default="0 0 0"/>
-	<xacro:arg name="mesh_suffix" default="stl"/>
-	<xacro:arg name="kinematics_suffix" default=""/>
-	<!-- load xarm device -->
+	<!-- load xarm6 device -->
 	<xacro:include filename="$(find xarm_description)/urdf/xarm_device_macro.xacro" />
-	<xacro:xarm_device prefix="$(arg prefix)" hw_ns="$(arg hw_ns)" limited="$(arg limited)"
-		effort_control="$(arg effort_control)" velocity_control="$(arg velocity_control)"
-		add_gripper="$(arg add_gripper)" add_vacuum_gripper="$(arg add_vacuum_gripper)"
-		add_bio_gripper="$(arg add_bio_gripper)" dof="$(arg dof)"
-		ros2_control_plugin="$(arg ros2_control_plugin)" robot_type="$(arg robot_type)"
-		load_gazebo_plugin="true" ros2_control_params="$(arg ros2_control_params)"
-		add_realsense_d435i="$(arg add_realsense_d435i)"
-		add_d435i_links="$(arg add_d435i_links)"
-		add_other_geometry="$(arg add_other_geometry)"
-		geometry_type="$(arg geometry_type)" geometry_mass="$(arg geometry_mass)"
-		geometry_height="$(arg geometry_height)" geometry_radius="$(arg geometry_radius)"
-		geometry_length="$(arg geometry_length)" geometry_width="$(arg geometry_width)"
-		geometry_mesh_filename="$(arg geometry_mesh_filename)"
-		geometry_mesh_origin_xyz="$(arg geometry_mesh_origin_xyz)" geometry_mesh_origin_rpy="$(arg geometry_mesh_origin_rpy)"
-		geometry_mesh_tcp_xyz="$(arg geometry_mesh_tcp_xyz)" geometry_mesh_tcp_rpy="$(arg geometry_mesh_tcp_rpy)"
-		robot_ip="$(arg robot_ip)" report_type="$(arg report_type)"
-		baud_checkset="$(arg baud_checkset)" default_gripper_baud="$(arg default_gripper_baud)"
-		model1300="$(arg model1300)" attach_to="$(arg attach_to)" attach_xyz="$(arg attach_xyz)" attach_rpy="$(arg attach_rpy)"
-		robot_sn="$(arg robot_sn)" use_gazebo_camera="$(arg use_gazebo_camera)" mesh_suffix="$(arg mesh_suffix)" kinematics_suffix="$(arg kinematics_suffix)" />
+	<xacro:xarm_device prefix="left" hw_ns="xarm" limited="false"
+		effort_control="false" velocity_control="false"
+		add_gripper="true" add_vacuum_gripper="false"
+		add_bio_gripper="false" dof="6"
+		ros2_control_plugin="uf_robot_hardware/UFRobotSystemHardware" robot_type="xarm"
+		load_gazebo_plugin="false" ros2_control_params=""
+		add_realsense_d435i="false"
+		add_d435i_links="true"
+		add_other_geometry="false"
+		geometry_type="box" geometry_mass="0.1"
+		geometry_height="0.1" geometry_radius="0.1"
+		geometry_length="0.1" geometry_width="0.1"
+		geometry_mesh_filename=""
+		geometry_mesh_origin_xyz="0 0 0" geometry_mesh_origin_rpy="0 0 0"
+		geometry_mesh_tcp_xyz="0 0 0" geometry_mesh_tcp_rpy="0 0 0"
+		robot_ip="192.168.1.210" report_type="dev"
+		baud_checkset="true" default_gripper_baud="2000000"
+		model1300="false" attach_to="left_arm_mount" attach_xyz="0 0 0" attach_rpy="0 0 0"
+		robot_sn="" use_gazebo_camera="false" mesh_suffix="stl" kinematics_suffix="" />
+	<xacro:xarm_device prefix="right" hw_ns="xarm" limited="false"
+		effort_control="false" velocity_control="false"
+		add_gripper="true" add_vacuum_gripper="false"
+		add_bio_gripper="false" dof="7"
+		ros2_control_plugin="uf_robot_hardware/UFRobotSystemHardware" robot_type="xarm"
+		load_gazebo_plugin="false" ros2_control_params=""
+		add_realsense_d435i="false"
+		add_d435i_links="true"
+		add_other_geometry="false"
+		geometry_type="box" geometry_mass="0.1"
+		geometry_height="0.1" geometry_radius="0.1"
+		geometry_length="0.1" geometry_width="0.1"
+		geometry_mesh_filename=""
+		geometry_mesh_origin_xyz="0 0 0" geometry_mesh_origin_rpy="0 0 0"
+		geometry_mesh_tcp_xyz="0 0 0" geometry_mesh_tcp_rpy="0 0 0"
+		robot_ip="192.168.1.211" report_type="dev"
+		baud_checkset="true" default_gripper_baud="2000000"
+		model1300="false" attach_to="right_arm_mount" attach_xyz="0 0 0" attach_rpy="0 0 0"
+		robot_sn="" use_gazebo_camera="false" mesh_suffix="stl" kinematics_suffix="" />
 </robot>

File: dim_cpp/urdf/include/alfred_base.urdf.xacro (robot description, xacro)
@@ -220,5 +220,5 @@
             <parent link="pillar_platform" />
             <child link="right_arm_mount" />
-            <origin xyz=".32675 -.319646 1.4125" rpy="-1.57079633 0 1.57079633" />
+            <origin xyz=".32675 -.319646 1.4125" rpy="1.57079633 3.14159265 1.57079633" />
         </joint>
     </xacro:macro>
