Commit message: Got dual xarm7 launch working with Alfred URDF

File: dim_cpp/urdf/alfred_base_descr.urdf.xacro (robot description, xacro)
@@ -1,7 +1,69 @@
 <?xml version="1.0"?>
 <robot name="alfred_base_descr" xmlns:xacro="http://ros.org/wiki/xacro">
+	<xacro:arg name="base_frame" default="world"/>
+	<xacro:arg name="prefix_1" default="L_"/>
+	<xacro:arg name="prefix_2" default="R_"/>
+	<xacro:arg name="hw_ns" default="xarm"/>
+	<xacro:arg name="limited" default="false"/>
+	<xacro:arg name="effort_control" default="false"/>
+	<xacro:arg name="velocity_control" default="false"/>
+	<xacro:arg name="add_gripper_1" default="true"/>
+	<xacro:arg name="add_gripper_2" default="true"/>
+	<xacro:arg name="add_vacuum_gripper_1" default="false"/>
+	<xacro:arg name="add_vacuum_gripper_2" default="false"/>
+	<xacro:arg name="add_bio_gripper_1" default="false"/>
+	<xacro:arg name="add_bio_gripper_2" default="false"/>
+	<xacro:arg name="model1300_1" default="false"/>
+	<xacro:arg name="model1300_2" default="false"/>
+	<xacro:arg name="dof_1" default="7"/>
+	<xacro:arg name="dof_2" default="7"/>
+	<xacro:arg name="robot_ip_1" default=""/>
+	<xacro:arg name="robot_ip_2" default=""/>
+	<xacro:arg name="robot_type_1" default="xarm"/>
+	<xacro:arg name="robot_type_2" default="xarm"/>
+	<xacro:arg name="robot_sn_1" default=""/>
+	<xacro:arg name="robot_sn_2" default=""/>
+	<xacro:arg name="report_type_1" default="normal"/>
+	<xacro:arg name="report_type_2" default="normal"/>
+	<xacro:arg name="ros2_control_plugin" default="uf_robot_hardware/UFFakeRobotSystemHardware"/>
+	<xacro:arg name="ros2_control_params" default=""/>
+	<xacro:arg name="add_realsense_d435i_1" default="false"/>
+	<xacro:arg name="add_realsense_d435i_2" default="false"/>
+	<xacro:arg name="add_d435i_links_1" default="true"/>
+	<xacro:arg name="add_d435i_links_2" default="true"/>
+	<xacro:arg name="add_other_geometry_1" default="false"/>
+	<xacro:arg name="geometry_type_1" default="box"/>
+	<xacro:arg name="geometry_mass_1" default="0.1"/>
+	<xacro:arg name="geometry_height_1" default="0.1"/>
+	<xacro:arg name="geometry_radius_1" default="0.1"/>
+	<xacro:arg name="geometry_length_1" default="0.1"/>
+	<xacro:arg name="geometry_width_1" default="0.1"/>
+	<xacro:arg name="geometry_mesh_filename_1" default=""/>
+	<xacro:arg name="geometry_mesh_origin_xyz_1" default="0 0 0"/>
+	<xacro:arg name="geometry_mesh_origin_rpy_1" default="0 0 0"/>
+	<xacro:arg name="geometry_mesh_tcp_xyz_1" default="0 0 0"/>
+	<xacro:arg name="geometry_mesh_tcp_rpy_1" default="0 0 0"/>
+	<xacro:arg name="add_other_geometry_2" default="false"/>
+	<xacro:arg name="geometry_type_2" default="box"/>
+	<xacro:arg name="geometry_mass_2" default="0.1"/>
+	<xacro:arg name="geometry_height_2" default="0.1"/>
+	<xacro:arg name="geometry_radius_2" default="0.1"/>
+	<xacro:arg name="geometry_length_2" default="0.1"/>
+	<xacro:arg name="geometry_width_2" default="0.1"/>
+	<xacro:arg name="geometry_mesh_filename_2" default=""/>
+	<xacro:arg name="geometry_mesh_origin_xyz_2" default="0 0 0"/>
+	<xacro:arg name="geometry_mesh_origin_rpy_2" default="0 0 0"/>
+	<xacro:arg name="geometry_mesh_tcp_xyz_2" default="0 0 0"/>
+	<xacro:arg name="geometry_mesh_tcp_rpy_2" default="0 0 0"/>
+	<xacro:arg name="baud_checkset_1" default="true"/>
+	<xacro:arg name="baud_checkset_2" default="true"/>
+	<xacro:arg name="default_gripper_baud_1" default="2000000"/>
+	<xacro:arg name="default_gripper_baud_2" default="2000000"/>
+	<xacro:arg name="mesh_suffix" default="stl"/>
+	<xacro:arg name="kinematics_suffix_1" default=""/>
+	<xacro:arg name="kinematics_suffix_2" default=""/>
 	<xacro:include filename="$(find dim_cpp)/urdf/include/alfred_base.urdf.xacro" />
-	<link name="local_world" />
-	<xacro:alfred_base base_frame="local_world" base_pos_x="0.0" base_pos_y="0.0" base_pos_z="0.0" base_roll="0.0" base_pitch="0.0" base_yaw="0.0" r="0.8" g="0.8" b="0.8" a="1.0" />
+	<link name="$(arg base_frame)" />
+	<xacro:alfred_base base_frame="$(arg base_frame)" base_pos_x="0.0" base_pos_y="0.0" base_pos_z="0.0" base_roll="0.0" base_pitch="0.0" base_yaw="0.0" r="0.8" g="0.8" b="0.8" a="1.0" />
 	<xacro:include filename="$(find depthai_descriptions)/urdf/include/depthai_macro.urdf.xacro" />
 	<xacro:depthai_camera camera_name="head_cam" parent="head_cam_link"
@@ -15,41 +77,41 @@
 	<!-- load xarm6 device -->
 	<xacro:include filename="$(find xarm_description)/urdf/xarm_device_macro.xacro" />
-	<xacro:xarm_device prefix="right_" hw_ns="xarm" limited="false"
-		effort_control="false" velocity_control="false"
-		add_gripper="true" add_vacuum_gripper="false"
-		add_bio_gripper="false" dof="7"
-		ros2_control_plugin="uf_robot_hardware/UFRobotFakeSystemHardware" robot_type="xarm"
-		load_gazebo_plugin="true" ros2_control_params=""
-		add_realsense_d435i="false"
-		add_d435i_links="true"
-		add_other_geometry="false"
-		geometry_type="box" geometry_mass="0.1"
-		geometry_height="0.1" geometry_radius="0.1"
-		geometry_length="0.1" geometry_width="0.1"
-		geometry_mesh_filename=""
-		geometry_mesh_origin_xyz="0 0 0" geometry_mesh_origin_rpy="0 0 0"
-		geometry_mesh_tcp_xyz="0 0 0" geometry_mesh_tcp_rpy="0 0 0"
-		robot_ip="192.168.1.197" report_type="dev"
-		baud_checkset="true" default_gripper_baud="2000000"
-		model1300="false" attach_to="right_arm_mount" attach_xyz="0 0 0" attach_rpy="0 0 0"
-		robot_sn="" use_gazebo_camera="false" mesh_suffix="stl" kinematics_suffix="" />
-	<xacro:xarm_device prefix="left_" hw_ns="xarm" limited="false"
-		effort_control="false" velocity_control="false"
-		add_gripper="true" add_vacuum_gripper="false"
-		add_bio_gripper="false" dof="6"
-		ros2_control_plugin="uf_robot_hardware/UFRobotFakeSystemHardware" robot_type="xarm"
-		load_gazebo_plugin="false" ros2_control_params=""
-		add_realsense_d435i="false"
-		add_d435i_links="true"
-		add_other_geometry="false"
-		geometry_type="box" geometry_mass="0.1"
-		geometry_height="0.1" geometry_radius="0.1"
-		geometry_length="0.1" geometry_width="0.1"
-		geometry_mesh_filename=""
-		geometry_mesh_origin_xyz="0 0 0" geometry_mesh_origin_rpy="0 0 0"
-		geometry_mesh_tcp_xyz="0 0 0" geometry_mesh_tcp_rpy="0 0 0"
-		robot_ip="192.168.1.210" report_type="dev"
-		baud_checkset="true" default_gripper_baud="2000000"
-		model1300="false" attach_to="left_arm_mount" attach_xyz="0 0 0" attach_rpy="0 0 0"
-		robot_sn="" use_gazebo_camera="false" mesh_suffix="stl" kinematics_suffix="" />
+	<xacro:xarm_device prefix="$(arg prefix_1)" hw_ns="$(arg hw_ns)" limited="$(arg limited)"
+		effort_control="$(arg effort_control)" velocity_control="$(arg velocity_control)"
+		add_gripper="$(arg add_gripper_1)" add_vacuum_gripper="$(arg add_vacuum_gripper_1)"
+		add_bio_gripper="$(arg add_bio_gripper_1)" dof="$(arg dof_1)"
+		ros2_control_plugin="$(arg ros2_control_plugin)" robot_type="$(arg robot_type_1)"
+		load_gazebo_plugin="false" ros2_control_params="$(arg ros2_control_params)"
+		attach_to="left_arm_mount" attach_xyz="0 0 0" attach_rpy="0 0 0"
+		add_realsense_d435i="$(arg add_realsense_d435i_1)"
+		add_d435i_links="$(arg add_d435i_links_1)"
+		add_other_geometry="$(arg add_other_geometry_1)"
+		geometry_type="$(arg geometry_type_1)" geometry_mass="$(arg geometry_mass_1)"
+		geometry_height="$(arg geometry_height_1)" geometry_radius="$(arg geometry_radius_1)"
+		geometry_length="$(arg geometry_length_1)" geometry_width="$(arg geometry_width_1)"
+		geometry_mesh_filename="$(arg geometry_mesh_filename_1)"
+		geometry_mesh_origin_xyz="$(arg geometry_mesh_origin_xyz_1)" geometry_mesh_origin_rpy="$(arg geometry_mesh_origin_rpy_1)"
+		geometry_mesh_tcp_xyz="$(arg geometry_mesh_tcp_xyz_1)" geometry_mesh_tcp_rpy="$(arg geometry_mesh_tcp_rpy_1)"
+		robot_ip="$(arg robot_ip_1)" report_type="$(arg report_type_1)"
+		baud_checkset="$(arg baud_checkset_1)" default_gripper_baud="$(arg default_gripper_baud_1)"
+		model1300="$(arg model1300_1)" robot_sn="$(arg robot_sn_1)" mesh_suffix="$(arg mesh_suffix)" kinematics_suffix="$(arg kinematics_suffix_1)" />
+	<xacro:xarm_device prefix="$(arg prefix_2)" hw_ns="$(arg hw_ns)" limited="$(arg limited)"
+		effort_control="$(arg effort_control)" velocity_control="$(arg velocity_control)"
+		add_gripper="$(arg add_gripper_2)" add_vacuum_gripper="$(arg add_vacuum_gripper_2)"
+		add_bio_gripper="$(arg add_bio_gripper_2)" dof="$(arg dof_2)"
+		ros2_control_plugin="$(arg ros2_control_plugin)" robot_type="$(arg robot_type_2)"
+		load_gazebo_plugin="true" ros2_control_params="$(arg ros2_control_params)"
+		attach_to="right_arm_mount" attach_xyz="0 0 0" attach_rpy="0 0 0"
+		add_realsense_d435i="$(arg add_realsense_d435i_2)"
+		add_d435i_links="$(arg add_d435i_links_2)"
+		add_other_geometry="$(arg add_other_geometry_2)"
+		geometry_type="$(arg geometry_type_2)" geometry_mass="$(arg geometry_mass_2)"
+		geometry_height="$(arg geometry_height_2)" geometry_radius="$(arg geometry_radius_2)"
+		geometry_length="$(arg geometry_length_2)" geometry_width="$(arg geometry_width_2)"
+		geometry_mesh_filename="$(arg geometry_mesh_filename_2)"
+		geometry_mesh_origin_xyz="$(arg geometry_mesh_origin_xyz_2)" geometry_mesh_origin_rpy="$(arg geometry_mesh_origin_rpy_2)"
+		geometry_mesh_tcp_xyz="$(arg geometry_mesh_tcp_xyz_2)" geometry_mesh_tcp_rpy="$(arg geometry_mesh_tcp_rpy_2)"
+		robot_ip="$(arg robot_ip_2)" report_type="$(arg report_type_2)"
+		baud_checkset="$(arg baud_checkset_2)" default_gripper_baud="$(arg default_gripper_baud_2)"
+		model1300="$(arg model1300_2)" robot_sn="$(arg robot_sn_2)" mesh_suffix="$(arg mesh_suffix)" kinematics_suffix="$(arg kinematics_suffix_2)" />
 </robot>

File: dim_cpp/urdf/include/alfred_base.urdf.xacro (robot description, xacro)
@@ -67,9 +67,14 @@
             </inertial>
         </link>
-        <joint name="right_wheel_joint" type="continuous">
+        <!-- <joint name="right_wheel_joint" type="continuous">
             <parent link="alfred_base_link" />
             <child link="botwheel_right" />
             <origin xyz="-0.0561 -0.395 -0.0375" rpy="0 0 -1.5707" />
             <axis xyz="0 1 0" />
+        </joint> -->
+        <joint name="right_wheel_joint" type="fixed">
+            <parent link="alfred_base_link" />
+            <child link="botwheel_right" />
+            <origin xyz="-0.0561 -0.395 -0.0375" rpy="0 0 -1.5707" />
         </joint>
         <link name="botwheel_left">
@@ -97,9 +102,14 @@
             </inertial>
         </link>
-        <joint name="left_wheel_joint" type="continuous">
+        <!-- <joint name="left_wheel_joint" type="continuous">
             <parent link="alfred_base_link" />
             <child link="botwheel_left" />
             <origin xyz="0.5061 -0.395 -0.0375" rpy="0 0 1.5707" />
             <axis xyz="0 1 0" />
+        </joint> -->
+        <joint name="left_wheel_joint" type="fixed">
+            <parent link="alfred_base_link" />
+            <child link="botwheel_left" />
+            <origin xyz="0.5061 -0.395 -0.0375" rpy="0 0 1.5707" />
         </joint>
         <link name="pillar_platform">
@@ -128,5 +138,5 @@
             </inertial>
         </link>
-        <joint name="pillar_platform_joint" type="prismatic">
+        <!-- <joint name="pillar_platform_joint" type="prismatic">
             <parent link="alfred_base_link" />
             <child link="pillar_platform" />
@@ -134,4 +144,9 @@
             <axis xyz="0 0 1" />
             <limit lower="-0.83" upper="0.0" effort="100" velocity="0.1"/>
+        </joint> -->
+        <joint name="pillar_platform_joint" type="fixed">
+            <parent link="alfred_base_link" />
+            <child link="pillar_platform" />
+            <origin xyz="0 0 0" rpy="0 0 0" />
         </joint>
         <link name="tilt_base">
@@ -159,5 +174,5 @@
             </inertial>
         </link>
-        <joint name="pan_joint" type="revolute">
+        <!-- <joint name="pan_joint" type="revolute">
             <parent link="alfred_base_link" />
             <child link="tilt_base" />
@@ -165,4 +180,9 @@
             <axis xyz="0 0 1"/>
             <limit lower="-1.57" upper="1.57" effort="100" velocity="0.1"/>
+        </joint> -->
+        <joint name="pan_joint" type="fixed">
+            <parent link="alfred_base_link" />
+            <child link="tilt_base" />
+            <origin xyz=".225 -.365 1.645" rpy="0 0 0" />
         </joint>
         <link name="camera_holder" >
@@ -191,5 +211,5 @@
             </inertial>
         </link>
-        <joint name="tilt_joint" type="revolute">
+        <!-- <joint name="tilt_joint" type="revolute">
             <parent link="tilt_base" />
             <child link="camera_holder" />
@@ -197,4 +217,9 @@
             <axis xyz="1 0 0" />
             <limit lower="-1.57" upper="1.57" effort="100" velocity="0.1"/>
+        </joint> -->
+        <joint name="tilt_joint" type="fixed">
+            <parent link="tilt_base" />
+            <child link="camera_holder" />
+            <origin xyz="0 0 0.014" rpy="0 0 0" />
         </joint>
         <link name="head_cam_link" />

Commit message: Odom updates with testing out topic based hardware interface

File: dim_cpp/urdf/alfred_base_descr.urdf.xacro (robot description, xacro)
@@ -116,5 +116,5 @@
 		model1300="$(arg model1300_2)" robot_sn="$(arg robot_sn_2)" mesh_suffix="$(arg mesh_suffix)" kinematics_suffix="$(arg kinematics_suffix_2)" />
 	<xacro:include filename="$(find dim_cpp)/urdf/alfred_wheels_ros2_control.xacro" />
-	<xacro:alfred_wheels_ros2_control />
+	<xacro:alfred_wheels_ros2_control mock_hardware="true"/>
 	<xacro:include filename="$(find dim_cpp)/urdf/alfred_pan_tilt_ros2_control.xacro" />
 	<xacro:alfred_pan_tilt_ros2_control />

File: dim_cpp/urdf/alfred_pan_tilt_ros2_control.xacro (robot description, xacro)
@@ -9,9 +9,13 @@
             <joint name="pan_joint">
                 <command_interface name="position"/>
-                <state_interface name="position"/>
+                <state_interface name="position">
+                    <param name="initial_value">0.0</param>
+                </state_interface>
             </joint>
             <joint name="tilt_joint">
                 <command_interface name="position"/>
-                <state_interface name="position"/>
+                <state_interface name="position">
+                    <param name="initial_value">0.0</param>
+                </state_interface>
             </joint>
         </ros2_control>

File: dim_cpp/urdf/alfred_wheels_ros2_control.xacro (robot description, xacro)
@@ -1,21 +1,58 @@
 <?xml version="1.0"?>
 <robot xmlns:xacro="http://www.ros.org/wiki/xacro">
-    <xacro:macro name="alfred_wheels_ros2_control" params="">
-        <ros2_control name="alfred_wheels" type="system">
-            <hardware>
-                <plugin>mock_components/GenericSystem</plugin>
-                <param name="calculate_dynamics">true</param>
-            </hardware>
-            <joint name="left_wheel_joint">
-                <command_interface name="velocity"/>
-                <state_interface name="position"/>
-                <state_interface name="velocity"/>
-            </joint>
-            <joint name="right_wheel_joint">
-                <command_interface name="velocity"/>
-                <state_interface name="position"/>
-                <state_interface name="velocity"/>
-            </joint>
-        </ros2_control>
+    <xacro:macro name="alfred_wheels_ros2_control" params="mock_hardware:=true">
+        <xacro:if value="${mock_hardware}">
+            <ros2_control name="alfred_wheels" type="system">
+                <hardware>
+                    <plugin>mock_components/GenericSystem</plugin>
+                    <param name="calculate_dynamics">true</param>
+                </hardware>
+                <joint name="left_wheel_joint">
+                    <command_interface name="velocity"/>
+                    <state_interface name="position">
+                        <param name="initial_value">0.0</param>
+                    </state_interface>
+                    <state_interface name="velocity">
+                        <param name="initial_value">0.0</param>
+                    </state_interface>
+                </joint>
+                <joint name="right_wheel_joint">
+                    <command_interface name="velocity"/>
+                    <state_interface name="position">
+                        <param name="initial_value">0.0</param>
+                    </state_interface>
+                    <state_interface name="velocity">
+                        <param name="initial_value">0.0</param>
+                    </state_interface>
+                </joint>
+            </ros2_control>
+        </xacro:if>
+        <xacro:unless value="${mock_hardware}">
+            <ros2_control name="alfred_wheels" type="system">
+                <hardware>
+                    <plugin>topic_based_ros2_control/TopicBasedSystem</plugin>
+                    <param name="joint_commands_topic">/alfred_wheels_commands</param>
+                    <param name="joint_states_topic">/alfred_wheels_states</param>
+                </hardware>
+                <joint name="left_wheel_joint">
+                    <command_interface name="velocity"/>
+                    <state_interface name="position">
+                        <param name="initial_value">0.0</param>
+                    </state_interface>
+                    <state_interface name="velocity">
+                        <param name="initial_value">0.0</param>
+                    </state_interface>
+                </joint>
+                <joint name="right_wheel_joint">
+                    <command_interface name="velocity"/>
+                    <state_interface name="position">
+                        <param name="initial_value">0.0</param>
+                    </state_interface>
+                    <state_interface name="velocity">
+                        <param name="initial_value">0.0</param>
+                    </state_interface>
+                </joint>
+            </ros2_control>
+        </xacro:unless>
     </xacro:macro>
 </robot>
