Commit message: Corrected Zed camera offset for URDF

File: dim_cpp/urdf/xarm_devkit_base_descr.urdf.xacro (robot description, xacro)
@@ -47,5 +47,4 @@
 	<xacro:include filename="$(find dim_cpp)/urdf/include/devkit_base.urdf.xacro" />
 	<xacro:include filename="$(find dim_cpp)/urdf/include/piper_angled_base.urdf.xacro" />
-	<xacro:include filename="$(find dim_cpp)/piper_description/urdf/piper_description_macro.xacro" />
 	<link name="$(arg base_frame)" />
 	<xacro:devkit_base base_frame="$(arg base_frame)" base_pos_x="0.0" base_pos_y="0.0" base_pos_z="0.23625" base_roll="0.0" base_pitch="0.0" base_yaw="0.0" r="0.8" g="0.8" b="0.8" a="1.0" />
@@ -75,5 +74,6 @@
 		<parent link="camera_center_link"/>
 		<child link="zed_camera_link"/>
-		<origin xyz="0 -.015 -.01325" rpy="0 0 1.5707" />
+		<origin xyz="0 -.0143 -.01325" rpy="0 0 1.5707" />
+		<!-- The back of the camera is at y = -0.0218 -->
     </joint>
 	<xacro:zed_camera name="$(arg camera_name)" model="$(arg camera_model)" custom_baseline="$(arg custom_baseline)" enable_gnss="$(arg enable_gnss)">
