Commit message: General cleanup and changing deps to dim_cpp in generated urdf

File: dim_cpp/urdf/xarm6_openft_gripper.urdf (robot description, URDF)
Before this commit: robot devkit_base_descr, 19 links, 18 joints
Links:
- link left_finger: geometry collision mesh filename=package://dim_cpp/meshes/gripper/xarm/left_finger.stl; visual mesh filename=package://dim_cpp/meshes/gripper/xarm/left_finger.stl
- link left_inner_knuckle: geometry collision mesh filename=package://dim_cpp/meshes/gripper/xarm/left_inner_knuckle.stl; visual mesh filename=package://dim_cpp/meshes/gripper/xarm/left_inner_knuckle.stl
- link left_outer_knuckle: geometry collision mesh filename=package://dim_cpp/meshes/gripper/xarm/left_outer_knuckle.stl; visual mesh filename=package://dim_cpp/meshes/gripper/xarm/left_outer_knuckle.stl
- link link1: geometry collision mesh filename=package://dim_cpp/meshes/xarm6/visual/link1.stl; visual mesh filename=package://dim_cpp/meshes/xarm6/visual/link1.stl
- link link2: geometry collision mesh filename=package://dim_cpp/meshes/xarm6/visual/link2.stl; visual mesh filename=package://dim_cpp/meshes/xarm6/visual/link2.stl
- link link3: geometry collision mesh filename=package://dim_cpp/meshes/xarm6/visual/link3.stl; visual mesh filename=package://dim_cpp/meshes/xarm6/visual/link3.stl
- link link4: geometry collision mesh filename=package://dim_cpp/meshes/xarm6/visual/link4.stl; visual mesh filename=package://dim_cpp/meshes/xarm6/visual/link4.stl
- link link5: geometry collision mesh filename=package://dim_cpp/meshes/xarm6/visual/link5.stl; visual mesh filename=package://dim_cpp/meshes/xarm6/visual/link5.stl
- link link6: geometry collision mesh filename=package://dim_cpp/meshes/end_tool/collision/end_tool.stl; visual mesh filename=package://dim_cpp/meshes/xarm6/visual/link6.stl
- link link_base: geometry collision mesh filename=package://dim_cpp/meshes/xarm6/visual/link_base.stl; visual mesh filename=package://dim_cpp/meshes/xarm6/visual/link_base.stl
- link right_finger: geometry collision mesh filename=package://dim_cpp/meshes/gripper/xarm/right_finger.stl; visual mesh filename=package://dim_cpp/meshes/gripper/xarm/right_finger.stl
- link right_inner_knuckle: geometry collision mesh filename=package://dim_cpp/meshes/gripper/xarm/right_inner_knuckle.s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; visual mesh filename=package://dim_cpp/meshes/gripper/xarm/right_inner_knuckle.s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
- link right_outer_knuckle: geometry collision mesh filename=package://dim_cpp/meshes/gripper/xarm/right_outer_knuckle.s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; visual mesh filename=package://dim_cpp/meshes/gripper/xarm/right_outer_knuckle.s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
- link xarm_gripper_base_link: geometry collision mesh filename=package://dim_cpp/meshes/gripper/xarm/base_link.stl; visual mesh filename=package://dim_cpp/meshes/gripper/xarm/base_link.stl

File: dim_cpp/urdf/xarm_openft_gripper.urdf.xacro (robot description, xacro)
@@ -1,4 +1,4 @@
 <?xml version="1.0"?>
-<robot name="devkit_base_descr"
+<robot name="xarm_openft_gripper"
 	xmlns:xacro="http://ros.org/wiki/xacro"
 	xmlns:drake="http://drake.mit.edu">
@@ -93,3 +93,8 @@
 		<origin rpy="0 0 1.570796" xyz="0 0 0.06"/>
 	</joint>
+	<drake:collision_filter_group name="no_collide">
+		<drake:member link="link_openft"/>
+		<drake:member link="xarm_gripper_base_link"/>
+		<drake:ignored_collision_filter_group name="no_collide"/>
+  </drake:collision_filter_group>
 </robot>
