Commit message: Added laser link

File: dim_cpp/urdf/include/alfred_base.urdf.xacro (robot description, xacro)
@@ -222,4 +222,10 @@
             <origin xyz=".32675 -.319646 1.4125" rpy="1.57079633 3.14159265 1.57079633" />
         </joint>
+        <link name="laser" />
+        <joint name="laser_joint" type="fixed">
+            <parent link="alfred_base_link" />
+            <child link="laser" />
+            <origin xyz=".225 .056557 .471777" rpy="0 0 -1.57079633" />
+        </joint>
     </xacro:macro>
     <!-- <xacro:alfred_base base_frame="world" base_pos_x="0.0" base_pos_y="0.0" base_pos_z="0.0" base_roll="0.0" base_pitch="0.0" base_yaw="0.0" r="0.8" g="0.8" b="0.8" a="1.0" /> -->

Commit message: Added SRDF for alfred base and got dual xarm launch working with it and fixed base joints

File: dim_cpp/urdf/include/alfred_base.urdf.xacro (robot description, xacro)
@@ -3,5 +3,5 @@
     xmlns:xacro="http://ros.org/wiki/xacro">
     <xacro:macro name="alfred_base"
-        params="base_frame  base_pos_x base_pos_y base_pos_z  base_roll base_pitch base_yaw r:=0.8 g:=0.8 b:=0.8 a:=1.0">
+        params="base_frame  base_pos_x base_pos_y base_pos_z  base_roll base_pitch base_yaw prefix:='' r:=0.8 g:=0.8 b:=0.8 a:=1.0 fixed:=true">
         <xacro:property
             name="file_prefix"
@@ -67,15 +67,19 @@
             </inertial>
         </link>
-        <!-- <joint name="right_wheel_joint" type="continuous">
-            <parent link="alfred_base_link" />
-            <child link="botwheel_right" />
-            <origin xyz="-0.0561 -0.395 -0.0375" rpy="0 0 -1.5707" />
-            <axis xyz="0 1 0" />
-        </joint> -->
-        <joint name="right_wheel_joint" type="fixed">
-            <parent link="alfred_base_link" />
-            <child link="botwheel_right" />
-            <origin xyz="-0.0561 -0.395 -0.0375" rpy="0 0 -1.5707" />
-        </joint>
+        <xacro:unless value="${fixed}">
+            <joint name="right_wheel_joint" type="continuous">
+                <parent link="alfred_base_link" />
+                <child link="botwheel_right" />
+                <origin xyz="-0.0561 -0.395 -0.0375" rpy="0 0 -1.5707" />
+                <axis xyz="0 1 0" />
+            </joint>
+        </xacro:unless>
+        <xacro:if value="${fixed}">
+            <joint name="right_wheel_joint" type="fixed">
+                <parent link="alfred_base_link" />
+                <child link="botwheel_right" />
+                <origin xyz="-0.0561 -0.395 -0.0375" rpy="0 0 -1.5707" />
+            </joint>
+        </xacro:if>
         <link name="botwheel_left">
             <visual>
@@ -102,15 +106,19 @@
             </inertial>
         </link>
-        <!-- <joint name="left_wheel_joint" type="continuous">
-            <parent link="alfred_base_link" />
-            <child link="botwheel_left" />
-            <origin xyz="0.5061 -0.395 -0.0375" rpy="0 0 1.5707" />
-            <axis xyz="0 1 0" />
-        </joint> -->
-        <joint name="left_wheel_joint" type="fixed">
-            <parent link="alfred_base_link" />
-            <child link="botwheel_left" />
-            <origin xyz="0.5061 -0.395 -0.0375" rpy="0 0 1.5707" />
-        </joint>
+        <xacro:unless value="${fixed}">
+            <joint name="left_wheel_joint" type="continuous">
+                <parent link="alfred_base_link" />
+                <child link="botwheel_left" />
+                <origin xyz="0.5061 -0.395 -0.0375" rpy="0 0 1.5707" />
+                <axis xyz="0 1 0" />
+            </joint>
+        </xacro:unless>
+        <xacro:if value="${fixed}">
+            <joint name="left_wheel_joint" type="fixed">
+                <parent link="alfred_base_link" />
+                <child link="botwheel_left" />
+                <origin xyz="0.5061 -0.395 -0.0375" rpy="0 0 1.5707" />
+            </joint>
+        </xacro:if>
         <link name="pillar_platform">
             <visual>
@@ -138,16 +146,20 @@
             </inertial>
         </link>
-        <!-- <joint name="pillar_platform_joint" type="prismatic">
-            <parent link="alfred_base_link" />
-            <child link="pillar_platform" />
-            <origin xyz="0 0 0" rpy="0 0 0" />
-            <axis xyz="0 0 1" />
-            <limit lower="-0.83" upper="0.0" effort="100" velocity="0.1"/>
-        </joint> -->
-        <joint name="pillar_platform_joint" type="fixed">
-            <parent link="alfred_base_link" />
-            <child link="pillar_platform" />
-            <origin xyz="0 0 0" rpy="0 0 0" />
-        </joint>
+        <xacro:unless value="${fixed}">
+            <joint name="pillar_platform_joint" type="prismatic">
+                <parent link="alfred_base_link" />
+                <child link="pillar_platform" />
+                <origin xyz="0 0 0" rpy="0 0 0" />
+                <axis xyz="0 0 1" />
+                <limit lower="-0.83" upper="0.0" effort="100" velocity="0.1"/>
+            </joint>
+        </xacro:unless>
+        <xacro:if value="${fixed}">
+            <joint name="pillar_platform_joint" type="fixed">
+                <parent link="alfred_base_link" />
+                <child link="pillar_platform" />
+                <origin xyz="0 0 0" rpy="0 0 0" />
+            </joint>
+        </xacro:if>
         <link name="tilt_base">
             <visual>
@@ -174,16 +186,20 @@
             </inertial>
         </link>
-        <!-- <joint name="pan_joint" type="revolute">
-            <parent link="alfred_base_link" />
-            <child link="tilt_base" />
-            <origin xyz=".225 -.365 1.645" rpy="0 0 0" />
-            <axis xyz="0 0 1"/>
-            <limit lower="-1.57" upper="1.57" effort="100" velocity="0.1"/>
-        </joint> -->
-        <joint name="pan_joint" type="fixed">
-            <parent link="alfred_base_link" />
-            <child link="tilt_base" />
-            <origin xyz=".225 -.365 1.645" rpy="0 0 0" />
-        </joint>
+        <xacro:unless value="${fixed}">
+            <joint name="pan_joint" type="revolute">
+                <parent link="alfred_base_link" />
+                <child link="tilt_base" />
+                <origin xyz=".225 -.365 1.645" rpy="0 0 0" />
+                <axis xyz="0 0 1"/>
+                <limit lower="-1.57" upper="1.57" effort="100" velocity="0.1"/>
+            </joint>
+        </xacro:unless>
+        <xacro:if value="${fixed}">
+            <joint name="pan_joint" type="fixed">
+                <parent link="alfred_base_link" />
+                <child link="tilt_base" />
+                <origin xyz=".225 -.365 1.645" rpy="0 0 0" />
+            </joint>
+        </xacro:if>
         <link name="camera_holder" >
             <visual>
@@ -211,16 +227,20 @@
             </inertial>
         </link>
-        <!-- <joint name="tilt_joint" type="revolute">
-            <parent link="tilt_base" />
-            <child link="camera_holder" />
-            <origin xyz="0 0 0.014" rpy="0 0 0" />
-            <axis xyz="1 0 0" />
-            <limit lower="-1.57" upper="1.57" effort="100" velocity="0.1"/>
-        </joint> -->
-        <joint name="tilt_joint" type="fixed">
-            <parent link="tilt_base" />
-            <child link="camera_holder" />
-            <origin xyz="0 0 0.014" rpy="0 0 0" />
-        </joint>
+        <xacro:unless value="${fixed}">
+            <joint name="tilt_joint" type="revolute">
+                <parent link="tilt_base" />
+                <child link="camera_holder" />
+                <origin xyz="0 0 0.014" rpy="0 0 0" />
+                <axis xyz="1 0 0" />
+                <limit lower="-1.57" upper="1.57" effort="100" velocity="0.1"/>
+            </joint>
+        </xacro:unless>
+        <xacro:if value="${fixed}">
+            <joint name="tilt_joint" type="fixed">
+                <parent link="tilt_base" />
+                <child link="camera_holder" />
+                <origin xyz="0 0 0.014" rpy="0 0 0" />
+            </joint>
+        </xacro:if>
         <link name="head_cam_link" />
         <joint name="head_cam_joint" type="fixed">

Commit message: Got navigation in rviz working with fixed URDF and control params. Also added auto launching of diff_drive controller

File: dim_cpp/urdf/include/alfred_base.urdf.xacro (robot description, xacro)
@@ -41,5 +41,5 @@
             <parent link="base_center" />
             <child link="alfred_base_link" />
-            <origin xyz="-.225 .2125 .1232" rpy="0 0 0" />
+            <origin xyz="-0.395 -.2125 .1232" rpy="0 0 1.5707" />
         </joint>
         <link name="botwheel_right">
@@ -111,5 +111,5 @@
                 <child link="botwheel_left" />
                 <origin xyz="0.5061 -0.395 -0.0375" rpy="0 0 1.5707" />
-                <axis xyz="0 1 0" />
+                <axis xyz="0 -1 0" />
             </joint>
         </xacro:unless>
