Commit message: Added custom gripper URDF, files, and controllers

File: dim_cpp/srdf/alfred_base_descr.srdf.xacro (robot description, xacro)
@@ -4,5 +4,5 @@
     <xacro:arg name="prefix_1" default="L_" />
     <xacro:arg name="prefix_2" default="R_" />
-    <xacro:arg name="dof_1" default="7" />
+    <xacro:arg name="dof_1" default="6" />
     <xacro:arg name="dof_2" default="7" />
     <xacro:arg name="robot_type_1" default="xarm" />
@@ -25,3 +25,10 @@
     <xacro:include filename="$(find dim_cpp)/srdf/alfred_base.srdf.xacro" />
     <xacro:alfred_base_macro_srdf />
+    <disable_collisions link1="$(arg prefix_1)gripper_base" link2="$(arg prefix_1)link$(arg dof_1)" reason="Never" />
+    <disable_collisions link1="$(arg prefix_2)gripper_base" link2="$(arg prefix_2)link$(arg dof_2)" reason="Never" />
+    <disable_collisions link1="$(arg prefix_1)gripper_base" link2="$(arg prefix_1)link_eef" reason="Adjacent" />
+    <disable_collisions link1="$(arg prefix_2)gripper_base" link2="$(arg prefix_2)link_eef" reason="Adjacent" />
+    <xacro:include filename="$(find dim_cpp)/srdf/alfred_gripper.srdf.xacro" />
+    <xacro:alfred_gripper_macro_srdf prefix="$(arg prefix_1)" />
+    <xacro:alfred_gripper_macro_srdf prefix="$(arg prefix_2)" />
 </robot>

File: dim_cpp/urdf/alfred_base_descr.urdf (robot description, URDF)
Before this commit: robot alfred_base_descr, 63 links, 62 joints
Links:
- removed link left_left_finger
- removed link left_left_inner_knuckle
- removed link left_left_outer_knuckle
- removed link left_link1
- removed link left_link2
- removed link left_link3
- removed link left_link4
- removed link left_link5
- removed link left_link6
- removed link left_link_base
- removed link left_link_eef
- removed link left_link_tcp
- removed link left_right_finger
- removed link left_right_inner_knuckle
- removed link left_right_outer_knuckle
- removed link left_xarm_gripper_base_link
- removed link local_world
- removed link right_left_finger
- removed link right_left_inner_knuckle
- removed link right_left_outer_knuckle
- removed link right_link1
- removed link right_link2
- removed link right_link3
- removed link right_link4
- removed link right_link5
- removed link right_link6
- removed link right_link7
- removed link right_link_base
- removed link right_link_eef
- removed link right_link_tcp
- removed link right_right_finger
- removed link right_right_inner_knuckle
- removed link right_right_outer_knuckle
- removed link right_xarm_gripper_base_link
- added link L_left_finger, mass 0.048304; collision mesh filename=package://dim_cpp/meshes/gripper/xarm/left_finger.stl; visual mesh filename=package://dim_cpp/meshes/gripper/xarm/left_finger.stl
- added link L_left_inner_knuckle, mass 0.0230125781256706; collision mesh filename=package://dim_cpp/meshes/gripper/xarm/left_inner_knuckle.stl; visual mesh filename=package://dim_cpp/meshes/gripper/xarm/left_inner_knuckle.stl
- added link L_left_outer_knuckle, mass 0.033618; collision mesh filename=package://dim_cpp/meshes/gripper/xarm/left_outer_knuckle.stl; visual mesh filename=package://dim_cpp/meshes/gripper/xarm/left_outer_knuckle.stl
- added link L_link1, mass 2.3814; collision mesh filename=package://dim_cpp/meshes/xarm6/visual/link1.stl; visual mesh filename=package://dim_cpp/meshes/xarm6/visual/link1.stl
- added link L_link2, mass 2.2675; collision mesh filename=package://dim_cpp/meshes/xarm6/visual/link2.stl; visual mesh filename=package://dim_cpp/meshes/xarm6/visual/link2.stl
- added link L_link3, mass 1.875; collision mesh filename=package://dim_cpp/meshes/xarm6/visual/link3.stl; visual mesh filename=package://dim_cpp/meshes/xarm6/visual/link3.stl
- added link L_link4, mass 1.3192; collision mesh filename=package://dim_cpp/meshes/xarm6/visual/link4.stl; visual mesh filename=package://dim_cpp/meshes/xarm6/visual/link4.stl
- added link L_link5, mass 1.33854; collision mesh filename=package://dim_cpp/meshes/xarm6/visual/link5.stl; visual mesh filename=package://dim_cpp/meshes/xarm6/visual/link5.stl
- added link L_link6, mass 0.17; collision mesh filename=package://dim_cpp/meshes/end_tool/collision/end_tool.stl; visual mesh filename=package://dim_cpp/meshes/xarm6/visual/link6.stl
- added link L_link_base, mass 2.7; collision mesh filename=package://dim_cpp/meshes/xarm6/visual/link_base.stl; visual mesh filename=package://dim_cpp/meshes/xarm6/visual/link_base.stl
- added link L_link_eef
- added link L_link_tcp
- added link L_right_finger, mass 0.048304; collision mesh filename=package://dim_cpp/meshes/gripper/xarm/right_finger.stl; visual mesh filename=package://dim_cpp/meshes/gripper/xarm/right_finger.stl
- added link L_right_inner_knuckle, mass 0.023013; collision mesh filename=package://dim_cpp/meshes/gripper/xarm/right_inner_knuckle.s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; visual mesh filename=package://dim_cpp/meshes/gripper/xarm/right_inner_knuckle.s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
- added link L_right_outer_knuckle, mass 0.033618; collision mesh filename=package://dim_cpp/meshes/gripper/xarm/right_outer_knuckle.s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; visual mesh filename=package://dim_cpp/meshes/gripper/xarm/right_outer_knuckle.s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
- added link L_xarm_gripper_base_link, mass 0.54156; collision mesh filename=package://dim_cpp/meshes/gripper/xarm/base_link.stl; visual mesh filename=package://dim_cpp/meshes/gripper/xarm/base_link.stl
- added link R_left_finger, mass 0.048304; collision mesh filename=package://dim_cpp/meshes/gripper/xarm/left_finger.stl; visual mesh filename=package://dim_cpp/meshes/gripper/xarm/left_finger.stl
- added link R_left_inner_knuckle, mass 0.0230125781256706; collision mesh filename=package://dim_cpp/meshes/gripper/xarm/left_inner_knuckle.stl; visual mesh filename=package://dim_cpp/meshes/gripper/xarm/left_inner_knuckle.stl
- added link R_left_outer_knuckle, mass 0.033618; collision mesh filename=package://dim_cpp/meshes/gripper/xarm/left_outer_knuckle.stl; visual mesh filename=package://dim_cpp/meshes/gripper/xarm/left_outer_knuckle.stl
- added link R_link1, mass 2.382; collision mesh filename=package://dim_cpp/meshes/xarm7/visual/link1.stl; visual mesh filename=package://dim_cpp/meshes/xarm7/visual/link1.stl
- added link R_link2, mass 1.869; collision mesh filename=package://dim_cpp/meshes/xarm7/visual/link2.stl; visual mesh filename=package://dim_cpp/meshes/xarm7/visual/link2.stl
- added link R_link3, mass 1.6383; collision mesh filename=package://dim_cpp/meshes/xarm7/visual/link3.stl; visual mesh filename=package://dim_cpp/meshes/xarm7/visual/link3.stl
- added link R_link4, mass 1.7269; collision mesh filename=package://dim_cpp/meshes/xarm7/visual/link4.stl; visual mesh filename=package://dim_cpp/meshes/xarm7/visual/link4.stl
- added link R_link5, mass 1.3203; collision mesh filename=package://dim_cpp/meshes/xarm7/visual/link5.stl; visual mesh filename=package://dim_cpp/meshes/xarm7/visual/link5.stl
- added link R_link6, mass 1.325; collision mesh filename=package://dim_cpp/meshes/xarm7/visual/link6.stl; visual mesh filename=package://dim_cpp/meshes/xarm7/visual/link6.stl
- added link R_link7, mass 0.17; collision mesh filename=package://dim_cpp/meshes/end_tool/collision/end_tool.stl; visual mesh filename=package://dim_cpp/meshes/xarm7/visual/link7.stl
- added link R_link_base, mass 0.88556; collision mesh filename=package://dim_cpp/meshes/xarm7/visual/link_base.stl; visual mesh filename=package://dim_cpp/meshes/xarm7/visual/link_base.stl
- added link R_link_eef
- added link R_link_tcp
- added link R_right_finger, mass 0.048304; collision mesh filename=package://dim_cpp/meshes/gripper/xarm/right_finger.stl; visual mesh filename=package://dim_cpp/meshes/gripper/xarm/right_finger.stl
- added link R_right_inner_knuckle, mass 0.023013; collision mesh filename=package://dim_cpp/meshes/gripper/xarm/right_inner_knuckle.s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; visual mesh filename=package://dim_cpp/meshes/gripper/xarm/right_inner_knuckle.s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
- added link R_right_outer_knuckle, mass 0.033618; collision mesh filename=package://dim_cpp/meshes/gripper/xarm/right_outer_knuckle.s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; visual mesh filename=package://dim_cpp/meshes/gripper/xarm/right_outer_knuckle.s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
- added link R_xarm_gripper_base_link, mass 0.54156; collision mesh filename=package://dim_cpp/meshes/gripper/xarm/base_link.stl; visual mesh filename=package://dim_cpp/meshes/gripper/xarm/base_link.stl
- added link laser
- added link world
- link chest_cam_model_origin: geometry visual mesh filename=package://dim_cpp/urdf/models/OAK-D-PRO.stl
- link head_cam_model_origin: geometry visual mesh filename=package://dim_cpp/urdf/models/OAK-D-PRO.stl
Joints:
- removed joint left_drive_joint
- removed joint left_gripper_fix
- removed joint left_joint1
- removed joint left_joint2
- removed joint left_joint3
- removed joint left_joint4
- removed joint left_joint5
- removed joint left_joint6
- removed joint left_joint_eef
- removed joint left_joint_tcp
- removed joint left_left_finger_joint
- removed joint left_left_inner_knuckle_joint
- removed joint left_right_finger_joint
- removed joint left_right_inner_knuckle_joint
- removed joint left_right_outer_knuckle_joint
- removed joint left_world_joint
- removed joint right_drive_joint
- removed joint right_gripper_fix
- removed joint right_joint1
- removed joint right_joint2
- removed joint right_joint3
- removed joint right_joint4
- removed joint right_joint5
- removed joint right_joint6
- removed joint right_joint7
- removed joint right_joint_eef
- removed joint right_joint_tcp
- removed joint right_left_finger_joint
- removed joint right_left_inner_knuckle_joint
- removed joint right_right_finger_joint
- removed joint right_right_inner_knuckle_joint
- removed joint right_right_outer_knuckle_joint
- removed joint right_world_joint
- added joint L_drive_joint: type revolute, parent L_xarm_gripper_base_link, child L_left_outer_knuckle, origin xyz=0 0.035 0.059098 rpy=0 0 0, axis 1 0 0, limit lower=0 upper=0.85 effort=50 velocity=2
- added joint L_gripper_fix: type fixed, parent L_link_eef, child L_xarm_gripper_base_link, origin xyz=0 0 0 rpy=0 0 0
- added joint L_joint1: type revolute, parent L_link_base, child L_link1, origin xyz=0 0 0.267 rpy=0 0 0, axis 0 0 1, limit lower=-6.283185307179586 upper=6.283185307179586 effort=50.0 velocity=3.14
- added joint L_joint2: type revolute, parent L_link1, child L_link2, origin xyz=0 0 0 rpy=-1.5708 0 0, axis 0 0 1, limit lower=-2.059 upper=2.0944 effort=50.0 velocity=3.14
- added joint L_joint3: type revolute, parent L_link2, child L_link3, origin xyz=0.0535 -0.2845 0 rpy=0 0 0, axis 0 0 1, limit lower=-3.927 upper=0.19198 effort=32.0 velocity=3.14
- added joint L_joint4: type revolute, parent L_link3, child L_link4, origin xyz=0.0775 0.3425 0 rpy=-1.5708 0 0, axis 0 0 1, limit lower=-6.283185307179586 upper=6.283185307179586 effort=32.0 velocity=3.14
- added joint L_joint5: type revolute, parent L_link4, child L_link5, origin xyz=0 0 0 rpy=1.5708 0 0, axis 0 0 1, limit lower=-1.69297 upper=3.141592653589793 effort=32.0 velocity=3.14
- added joint L_joint6: type revolute, parent L_link5, child L_link6, origin xyz=0.076 0.097 0 rpy=-1.5708 0 0, axis 0 0 1, limit lower=-6.283185307179586 upper=6.283185307179586 effort=20.0 velocity=3.14
- added joint L_joint_eef: type fixed, parent L_link6, child L_link_eef, origin xyz=0 0 0 rpy=0 0 0
- added joint L_joint_tcp: type fixed, parent L_xarm_gripper_base_link, child L_link_tcp, origin xyz=0 0 0.172 rpy=0 0 0
- added joint L_left_finger_joint: type revolute, parent L_left_outer_knuckle, child L_left_finger, origin xyz=0 0.035465 0.042039 rpy=0 0 0, axis -1 0 0, limit lower=0 upper=0.85 effort=50 velocity=2, mimic joint=L_drive_joint multiplier=1 offset=0
- added joint L_left_inner_knuckle_joint: type revolute, parent L_xarm_gripper_base_link, child L_left_inner_knuckle, origin xyz=0 0.02 0.074098 rpy=0 0 0, axis 1 0 0, limit lower=0 upper=0.85 effort=50 velocity=2, mimic joint=L_drive_joint multiplier=1 offset=0
- added joint L_right_finger_joint: type revolute, parent L_right_outer_knuckle, child L_right_finger, origin xyz=0 -0.035465 0.042039 rpy=0 0 0, axis 1 0 0, limit lower=0 upper=0.85 effort=50 velocity=2, mimic joint=L_drive_joint multiplier=1 offset=0
- added joint L_right_inner_knuckle_joint: type revolute, parent L_xarm_gripper_base_link, child L_right_inner_knuckle, origin xyz=0 -0.02 0.074098 rpy=0 0 0, axis -1 0 0, limit lower=0 upper=0.85 effort=50 velocity=2, mimic joint=L_drive_joint multiplier=1 offset=0
- added joint L_right_outer_knuckle_joint: type revolute, parent L_xarm_gripper_base_link, child L_right_outer_knuckle, origin xyz=0 -0.035 0.059098 rpy=0 0 0, axis -1 0 0, limit lower=0 upper=0.85 effort=50 velocity=2, mimic joint=L_drive_joint multiplier=1 offset=0
- added joint L_world_joint: type fixed, parent left_arm_mount, child L_link_base, origin xyz=0 0 0 rpy=0 0 0
- added joint R_drive_joint: type revolute, parent R_xarm_gripper_base_link, child R_left_outer_knuckle, origin xyz=0 0.035 0.059098 rpy=0 0 0, axis 1 0 0, limit lower=0 upper=0.85 effort=50 velocity=2
- added joint R_gripper_fix: type fixed, parent R_link_eef, child R_xarm_gripper_base_link, origin xyz=0 0 0 rpy=0 0 0
- added joint R_joint1: type revolute, parent R_link_base, child R_link1, origin xyz=0 0 0.267 rpy=0 0 0, axis 0 0 1, limit lower=-6.283185307179586 upper=6.283185307179586 effort=50 velocity=3.14
- added joint R_joint2: type revolute, parent R_link1, child R_link2, origin xyz=0 0 0 rpy=-1.5708 0 0, axis 0 0 1, limit lower=-2.059 upper=2.0944 effort=50 velocity=3.14
- added joint R_joint3: type revolute, parent R_link2, child R_link3, origin xyz=0 -0.293 0 rpy=1.5708 0 0, axis 0 0 1, limit lower=-6.283185307179586 upper=6.283185307179586 effort=30 velocity=3.14
- added joint R_joint4: type revolute, parent R_link3, child R_link4, origin xyz=0.0525 0 0 rpy=1.5708 0 0, axis 0 0 1, limit lower=-0.19198 upper=3.927 effort=30 velocity=3.14
- added joint R_joint5: type revolute, parent R_link4, child R_link5, origin xyz=0.0775 -0.3425 0 rpy=1.5708 0 0, axis 0 0 1, limit lower=-6.283185307179586 upper=6.283185307179586 effort=30 velocity=3.14
- added joint R_joint6: type revolute, parent R_link5, child R_link6, origin xyz=0 0 0 rpy=1.5708 0 0, axis 0 0 1, limit lower=-1.69297 upper=3.141592653589793 effort=20 velocity=3.14
- added joint R_joint7: type revolute, parent R_link6, child R_link7, origin xyz=0.076 0.097 0 rpy=-1.5708 0 0, axis 0 0 1, limit lower=-6.283185307179586 upper=6.283185307179586 effort=20 velocity=3.14
- added joint R_joint_eef: type fixed, parent R_link7, child R_link_eef, origin xyz=0 0 0 rpy=0 0 0
- added joint R_joint_tcp: type fixed, parent R_xarm_gripper_base_link, child R_link_tcp, origin xyz=0 0 0.172 rpy=0 0 0
- added joint R_left_finger_joint: type revolute, parent R_left_outer_knuckle, child R_left_finger, origin xyz=0 0.035465 0.042039 rpy=0 0 0, axis -1 0 0, limit lower=0 upper=0.85 effort=50 velocity=2, mimic joint=R_drive_joint multiplier=1 offset=0
- added joint R_left_inner_knuckle_joint: type revolute, parent R_xarm_gripper_base_link, child R_left_inner_knuckle, origin xyz=0 0.02 0.074098 rpy=0 0 0, axis 1 0 0, limit lower=0 upper=0.85 effort=50 velocity=2, mimic joint=R_drive_joint multiplier=1 offset=0
- added joint R_right_finger_joint: type revolute, parent R_right_outer_knuckle, child R_right_finger, origin xyz=0 -0.035465 0.042039 rpy=0 0 0, axis 1 0 0, limit lower=0 upper=0.85 effort=50 velocity=2, mimic joint=R_drive_joint multiplier=1 offset=0
- added joint R_right_inner_knuckle_joint: type revolute, parent R_xarm_gripper_base_link, child R_right_inner_knuckle, origin xyz=0 -0.02 0.074098 rpy=0 0 0, axis -1 0 0, limit lower=0 upper=0.85 effort=50 velocity=2, mimic joint=R_drive_joint multiplier=1 offset=0
- added joint R_right_outer_knuckle_joint: type revolute, parent R_xarm_gripper_base_link, child R_right_outer_knuckle, origin xyz=0 -0.035 0.059098 rpy=0 0 0, axis -1 0 0, limit lower=0 upper=0.85 effort=50 velocity=2, mimic joint=R_drive_joint multiplier=1 offset=0
- added joint R_world_joint: type fixed, parent right_arm_mount, child R_link_base, origin xyz=0 0 0 rpy=0 0 0
- added joint laser_joint: type fixed, parent alfred_base_link, child laser, origin xyz=.225 .056557 .471777 rpy=0 0 -1.57079633
- joint base_center_joint: origin xyz=-.225 .2125 .1232 rpy=0 0 0 -> xyz=-0.395 -.2125 .1232 rpy=0 0 1.5707
- joint base_parent_joint: parent local_world -> world
- joint left_wheel_joint: axis 0 1 0 -> 0 -1 0

File: dim_cpp/urdf/alfred_base_descr.urdf.xacro (robot description, xacro)
@@ -8,6 +8,6 @@
 	<xacro:arg name="effort_control" default="false"/>
 	<xacro:arg name="velocity_control" default="false"/>
-	<xacro:arg name="add_gripper_1" default="true"/>
-	<xacro:arg name="add_gripper_2" default="true"/>
+	<xacro:arg name="add_gripper_1" default="false"/>
+	<xacro:arg name="add_gripper_2" default="false"/>
 	<xacro:arg name="add_vacuum_gripper_1" default="false"/>
 	<xacro:arg name="add_vacuum_gripper_2" default="false"/>
@@ -64,4 +64,5 @@
 	<xacro:arg name="kinematics_suffix_2" default=""/>
 	<xacro:include filename="$(find dim_cpp)/urdf/include/alfred_base.urdf.xacro" />
+	<xacro:include filename="$(find dim_cpp)/urdf/include/alfred_gripper.urdf.xacro" />
 	<link name="$(arg base_frame)" />
 	<xacro:alfred_base base_frame="$(arg base_frame)" base_pos_x="0.0" base_pos_y="0.0" base_pos_z="0.0" base_roll="0.0" base_pitch="0.0" base_yaw="0.0" r="0.8" g="0.8" b="0.8" a="1.0" />
@@ -115,4 +116,6 @@
 		baud_checkset="$(arg baud_checkset_2)" default_gripper_baud="$(arg default_gripper_baud_2)"
 		model1300="$(arg model1300_2)" robot_sn="$(arg robot_sn_2)" mesh_suffix="$(arg mesh_suffix)" kinematics_suffix="$(arg kinematics_suffix_2)" />
+	<xacro:alfred_gripper prefix="$(arg prefix_1)" attach_to="L_link_eef" />
+	<xacro:alfred_gripper prefix="$(arg prefix_2)" attach_to="R_link_eef" />
 	<xacro:include filename="$(find dim_cpp)/urdf/alfred_wheels_ros2_control.xacro" />
 	<xacro:alfred_wheels_ros2_control mock_hardware="true"/>
@@ -121,3 +124,6 @@
 	<xacro:include filename="$(find dim_cpp)/urdf/alfred_pillar_platform_ros2_control.xacro" />
 	<xacro:alfred_pillar_platform_ros2_control />
+	<xacro:include filename="$(find dim_cpp)/urdf/alfred_gripper_ros2_control.xacro" />
+	<xacro:alfred_gripper_ros2_control prefix="$(arg prefix_1)" />
+	<xacro:alfred_gripper_ros2_control prefix="$(arg prefix_2)" />
 </robot>

File: xarm_ros2/xarm_moveit_config/srdf/alfred_base_descr.srdf.xacro (robot description, xacro)
@@ -25,3 +25,10 @@
     <xacro:include filename="$(find dim_cpp)/srdf/alfred_base.srdf.xacro" />
     <xacro:alfred_base_macro_srdf />
+    <disable_collisions link1="$(arg prefix_1)gripper_base" link2="$(arg prefix_1)link$(arg dof_1)" reason="Never" />
+    <disable_collisions link1="$(arg prefix_2)gripper_base" link2="$(arg prefix_2)link$(arg dof_2)" reason="Never" />
+    <disable_collisions link1="$(arg prefix_1)gripper_base" link2="$(arg prefix_1)link_eef" reason="Adjacent" />
+    <disable_collisions link1="$(arg prefix_2)gripper_base" link2="$(arg prefix_2)link_eef" reason="Adjacent" />
+    <xacro:include filename="$(find dim_cpp)/srdf/alfred_gripper.srdf.xacro" />
+    <xacro:alfred_gripper_macro_srdf prefix="$(arg prefix_1)" />
+    <xacro:alfred_gripper_macro_srdf prefix="$(arg prefix_2)" />
 </robot>
