Commit message: Added SRDF for custom gripper and added USD files for Isaac Sim

File: dim_cpp/srdf/alfred_gripper.srdf.xacro (robot description, xacro)
@@ -18,8 +18,9 @@
         </group_state>
         <group_state name="${prefix}gripper_close" group="${prefix}alfred_gripper">
-            <joint name="${prefix}jaw_1_joint" value="0.05" />
+            <joint name="${prefix}jaw_1_joint" value="0.04" />
         </group_state>
         <disable_collisions link1="${prefix}gripper_jaw_1" link2="${prefix}gripper_base" reason="Adjacent" />
         <disable_collisions link1="${prefix}gripper_jaw_2" link2="${prefix}gripper_base" reason="Adjacent" />
+        <disable_collisions link1="${prefix}gripper_jaw_1" link2="${prefix}gripper_jaw_2" reason="Adjacent" />
     </xacro:macro>
 </robot>

File: dim_cpp/urdf/alfred_base_descr.urdf (robot description, URDF)
Before this commit: robot alfred_base_descr, 64 links, 63 joints
Links:
- removed link L_left_finger
- removed link L_left_inner_knuckle
- removed link L_left_outer_knuckle
- removed link L_link_tcp
- removed link L_right_finger
- removed link L_right_inner_knuckle
- removed link L_right_outer_knuckle
- removed link L_xarm_gripper_base_link
- removed link R_left_finger
- removed link R_left_inner_knuckle
- removed link R_left_outer_knuckle
- removed link R_link_tcp
- removed link R_right_finger
- removed link R_right_inner_knuckle
- removed link R_right_outer_knuckle
- removed link R_xarm_gripper_base_link
- added link L_gripper_base, mass 0.5; collision mesh filename=package://dim_cpp/urdf/meshes/alfred_gripper_base-collision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 scale=0.001 0.001 0.001; visual mesh filename=package://dim_cpp/urdf/meshes/alfred_gripper_base-visual.stl scale=0.001 0.001 0.001
- added link L_gripper_jaw_1, mass 0.1; collision mesh filename=package://dim_cpp/urdf/meshes/alfred_gripper_jaw-collision.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 scale=0.001 0.001 0.001; visual mesh filename=package://dim_cpp/urdf/meshes/alfred_gripper_jaw-visual.stl scale=0.001 0.001 0.001
- added link L_gripper_jaw_2, mass 0.1; collision mesh filename=package://dim_cpp/urdf/meshes/alfred_gripper_jaw-collision.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 scale=0.001 0.001 0.001; visual mesh filename=package://dim_cpp/urdf/meshes/alfred_gripper_jaw-visual.stl scale=0.001 0.001 0.001
- added link R_gripper_base, mass 0.5; collision mesh filename=package://dim_cpp/urdf/meshes/alfred_gripper_base-collision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 scale=0.001 0.001 0.001; visual mesh filename=package://dim_cpp/urdf/meshes/alfred_gripper_base-visual.stl scale=0.001 0.001 0.001
- added link R_gripper_jaw_1, mass 0.1; collision mesh filename=package://dim_cpp/urdf/meshes/alfred_gripper_jaw-collision.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 scale=0.001 0.001 0.001; visual mesh filename=package://dim_cpp/urdf/meshes/alfred_gripper_jaw-visual.stl scale=0.001 0.001 0.001
- added link R_gripper_jaw_2, mass 0.1; collision mesh filename=package://dim_cpp/urdf/meshes/alfred_gripper_jaw-collision.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 scale=0.001 0.001 0.001; visual mesh filename=package://dim_cpp/urdf/meshes/alfred_gripper_jaw-visual.stl scale=0.001 0.001 0.001
Joints:
- removed joint L_drive_joint
- removed joint L_gripper_fix
- removed joint L_joint_tcp
- removed joint L_left_finger_joint
- removed joint L_left_inner_knuckle_joint
- removed joint L_right_finger_joint
- removed joint L_right_inner_knuckle_joint
- removed joint L_right_outer_knuckle_joint
- removed joint R_drive_joint
- removed joint R_gripper_fix
- removed joint R_joint_tcp
- removed joint R_left_finger_joint
- removed joint R_left_inner_knuckle_joint
- removed joint R_right_finger_joint
- removed joint R_right_inner_knuckle_joint
- removed joint R_right_outer_knuckle_joint
- added joint L_gripper_base_joint: type fixed, parent L_link_eef, child L_gripper_base, origin xyz=0 0 0.05 rpy=0 0 1.5707
- added joint L_jaw_1_joint: type prismatic, parent L_gripper_base, child L_gripper_jaw_1, origin xyz=0 0 0 rpy=0 0 0, axis 1 0 0, limit lower=0 upper=0.05 effort=100 velocity=0.1
- added joint L_jaw_2_joint: type prismatic, parent L_gripper_base, child L_gripper_jaw_2, origin xyz=0 0 0 rpy=0 0 3.14159, axis 1 0 0, limit lower=0 upper=0.05 effort=100 velocity=0.1, mimic joint=L_jaw_1_joint multiplier=1 offset=0
- added joint R_gripper_base_joint: type fixed, parent R_link_eef, child R_gripper_base, origin xyz=0 0 0.05 rpy=0 0 1.5707
- added joint R_jaw_1_joint: type prismatic, parent R_gripper_base, child R_gripper_jaw_1, origin xyz=0 0 0 rpy=0 0 0, axis 1 0 0, limit lower=0 upper=0.05 effort=100 velocity=0.1
- added joint R_jaw_2_joint: type prismatic, parent R_gripper_base, child R_gripper_jaw_2, origin xyz=0 0 0 rpy=0 0 3.14159, axis 1 0 0, limit lower=0 upper=0.05 effort=100 velocity=0.1, mimic joint=R_jaw_1_joint multiplier=1 offset=0
